File: PCB/BoostBuck.kicad_sch (KiCad schematic)
At the start: 15 parts, among them IC1 ABXS005A4X341-SRZ, J2 NID35-5, Q1 NPN

Commit message: comment
Other:
- note added: "Archi chelou!! Devraient être en parallèles et pas en série!"
Changed lines of the file:
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@@
+		)
+	)
+	(text "Archi chelou!!\nDevraient être en parallèles et pas en série!\n"
+		(exclude_from_sim no)
+		(at 42.926 54.864 0)
+		(effects
+			(font
+				(size 1.27 1.27)
+			)
 		)
 	)
@@
 		(effects
 			(font
+				(size 1.27 1.27)
+			)
+		)
+	)
+	(text "Archi chelou!!\nDevraient être en parallèles et pas en série!\n"
+		(exclude_from_sim no)
+		(at 119.38 51.816 0)
+		(effects
+			(font

Commit message: Add: Ethernet
Changed lines of the file:
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@@
 	(text "To have 24V"
 		(exclude_from_sim no)
-		(at 46.482 96.012 0)
+		(at 40.64 96.266 0)
 		(effects
 			(font
