File: PCB/Power.kicad_sch (KiCad schematic)
At the start: 0 parts

Commit message: ADD supplies to UC
Parts:
- added C56, C57, C58, C59, C60, C61, C62, C63, C64, C65, C66, C67, C68, C69, C70: 100n, symbol Device:C
- added C71: 4.7u, symbol Device:C
Connections:
- new net 3V3: C56.1, C57.1, C58.1, C59.1, C60.1, C61.1, C62.1, C63.1, C64.1, C65.1, C66.1, C67.1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
- new net GND: C56.2, C57.2, C58.2, C59.2, C60.2, C61.2, C62.2, C63.2, C64.2, C65.2, C66.2, C67.2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
Other:
- note added: "Must be as close as possible from µC"
