File: PCB/GPIO.kicad_sch (KiCad schematic)
At the start: 2 parts, among them J4 Conn_02x36_Counter_Clockwise, J5 Conn_02x36_Counter_Clockwise

Commit message: ADD: GPIO
Connections:
- net PF1: now also J5.69 (Pin_69)
- net PF11: now also J5.64 (Pin_64)
- net PF13: now also J5.63 (Pin_63)
- net PF15: now also J5.62 (Pin_62)
- net PF3: now also J5.68 (Pin_68)
- net PF5: now also J5.67 (Pin_67)
- net PF7: now also J5.66 (Pin_66)
- net PF9: now also J5.65 (Pin_65)
- net PG1: now also J5.61 (Pin_61)
- net PG11: now also J5.56 (Pin_56)
- net PG13: now also J5.55 (Pin_55)
- net PG15: now also J5.54 (Pin_54)
- net PG3: now also J5.60 (Pin_60)
- net PG5: now also J5.59 (Pin_59)
- net PG7: now also J5.58 (Pin_58)
- net PG9: now also J5.57 (Pin_57)
- net PH1: now also J5.53 (Pin_53)
- net PH11: now also J5.48 (Pin_48)
- net PH13: now also J5.47 (Pin_47)
- net PH15: now also J5.46 (Pin_46)
- net PH3: now also J5.52 (Pin_52)
- net PH5: now also J5.51 (Pin_51)
- net PH7: now also J5.50 (Pin_50)
- net PH9: now also J5.49 (Pin_49)
- net PI1: now also J5.45 (Pin_45)
- net PI11: now also J5.40 (Pin_40)
- net PI3: now also J5.44 (Pin_44)
- net PI5: now also J5.43 (Pin_43)
- net PI7: now also J5.42 (Pin_42)
- net PI9: now also J5.41 (Pin_41)

Commit message: Updated MCU sheet
Added decoupling capacitors
Linked Ethernet to MCU
Started Usb linking to MCU
Connections:
- net PH0: no longer names the net of J5.20 (Pin_20)
- net PH1: no longer names the net of J5.53 (Pin_53)
- no-connect marks 0 -> 4
Changed lines of the file:
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@@
 		)
 	)
+	(no_connect
+		(at 144.78 90.17)
+	)
+	(no_connect
+		(at 207.01 78.74)
+	)
+	(no_connect
+		(at 219.71 78.74)
+	)
+	(no_connect
+		(at 144.78 87.63)
+	)
 	(bus_entry
 		(at 148.59 41.91)
@@
 		)
 	)
-	(label "PH1"
-		(at 219.71 78.74 0)
-		(effects
-			(font
-				(size 1.27 1.27)
-			)
-			(justify left bottom)
-		)
-	)
 	(label "PD1"
 		(at 82.55 86.36 0)
@@
 		)
 	)
-	(label "PH0"
-		(at 207.01 78.74 180)
-		(effects
-			(font
-				(size 1.27 1.27)
-			)
-			(justify right bottom)
-		)
-	)
 	(label "PA13"
 		(at 69.85 71.12 180)
@@
 		)
 	)
-	(label "PH0"
-		(at 144.78 87.63 180)
-		(effects
-			(font
-				(size 1.27 1.27)
-			)
-			(justify right bottom)
-		)
-	)
 	(label "PC6"
 		(at 166.37 46.99 180)
@@
 		)
 	)
-	(label "PH1"
-		(at 144.78 90.17 180)
-		(effects
-			(font
-				(size 1.27 1.27)
-			)
-			(justify right bottom)
-		)
-	)
 	(label "PG10"
 		(at 207.01 71.12 180)
@@
 		)
 	)
-	(hierarchical_label "PH[0..15]"
+	(hierarchical_label "PH[2..15]"
 		(shape bidirectional)
 		(at 148.59 81.28 180)
