File: PCB/MCU_Debug.kicad_sch (KiCad schematic)
At the start: 0 parts

Commit message: Updated a lot of stuff:
Added encoders,
Added 5V power supply for actuators
Added 12V power supply for actuators
Renamed sheets to be clearer
Added usb debug
Modify MCU sheet to be A3 format
Linked some pins
Parts:
- added C76: 4.7nF, Capacitor_SMD:C_0603_1608Metric_Pad1.08x0.95mm_HandSolder, symbol Device:C
- added C77: 0.1uF, Capacitor_SMD:C_0603_1608Metric_Pad1.08x0.95mm_HandSolder, symbol Device:C
- added C78: 10nF, Capacitor_SMD:C_0603_1608Metric_Pad1.08x0.95mm_HandSolder, symbol Device:C
- added D2: LED_GREEN, LED_SMD:LED_0603_1608Metric, symbol Device:LED
- added D8: LED_RED, LED_SMD:LED_0603_1608Metric, symbol Device:LED
- added J11: USB_B_Micro, SamacSys_Parts:USB_Micro-B_Molex_47346-0001, symbol Connector:USB_B_Micro
- added R39: 400R, Resistor_SMD:R_0603_1608Metric, symbol Device:R
- added R40: 549R, Resistor_SMD:R_0603_1608Metric, symbol Device:R
- added R60: 1Meg, Resistor_SMD:R_0603_1608Metric_Pad0.98x0.95mm_HandSolder, symbol Device:R
- added U5: FT230XS, Package_SO:SSOP-16_3.9x4.9mm_P0.635mm, symbol Interface_USB:FT230XS
Connections:
- new net: D8.1 (K), R40.2
- new net: C76.1, J11.6 (Shield), R60.2
- new net: D2.1 (K), R39.2
- new net: J11.2 (D-), U5.9 (USBDM)
- new net: J11.3 (D+), U5.8 (USBDP)
- new net: R40.1, U5.7 (CBUS2)
- new net: R39.1, U5.14 (CBUS1)
- new net 3V3: C77.1, D2.2 (A), D8.2 (A), U5.10 (3V3OUT), U5.3 (VCCIO)
- new net 5V_DEBUG: C78.1, J11.1 (VBUS), U5.12 (VCC)
- new net GND: C76.2, C77.2, C78.2, J11.5 (GND), R60.1, U5.13 (GND), U5.5 (GND)
- new net NRST: U5.11 (~{RESET})
- new net RX_DEBUG: U5.4 (RXD)
- new net TX_DEBUG: U5.1 (TXD)
- no-connect marks 0 -> 5
Other:
- note added: "RXLED"
- note added: "TXLED"
