File: PCB/Power_Boost_24V.kicad_sch (KiCad schematic)
At the start: 31 parts, among them IC1 ABXS005A4X341-SRZ, Q1 BSS138, U3 125700D00000G, U4 125700D00000G

Commit message: Updated a lot of stuff:
Added encoders,
Added 5V power supply for actuators
Added 12V power supply for actuators
Renamed sheets to be clearer
Added usb debug
Modify MCU sheet to be A3 format
Linked some pins
Parts:
- R5: value 47k -> 100k
Connections:
- net 24V renamed OUT
- net GPIO_ENABLE renamed GPIO_ENABLE_24V
- net IN_24V renamed IN
Changed lines of the file:
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@@
 	(wire
 		(pts
-			(xy 250.19 22.86) (xy 256.54 22.86)
+			(xy 36.83 17.78) (xy 30.48 17.78)
 		)
 		(stroke
@@
 	)
 	(label "GPIO_ENABLE"
-		(at 250.19 22.86 180)
-		(effects
-			(font
-				(size 1.27 1.27)
-			)
-			(justify right bottom)
+		(at 36.83 17.78 0)
+		(effects
+			(font
+				(size 1.27 1.27)
+			)
+			(justify left bottom)
 		)
 	)
@@
 		)
 	)
-	(hierarchical_label "24V"
+	(hierarchical_label "OUT"
 		(shape output)
 		(at 256.54 30.48 0)
@@
 		)
 	)
-	(hierarchical_label "GPIO_ENABLE"
-		(shape output)
-		(at 256.54 22.86 0)
-		(effects
-			(font
-				(size 1.27 1.27)
-			)
-			(justify left)
-		)
-	)
-	(hierarchical_label "IN_24V"
+	(hierarchical_label "GPIO_ENABLE_24V"
+		(shape input)
+		(at 30.48 17.78 180)
+		(effects
+			(font
+				(size 1.27 1.27)
+			)
+			(justify right)
+		)
+	)
+	(hierarchical_label "IN"
 		(shape input)
 		(at 30.48 22.86 180)
@@
 			)
 		)
-		(property "Value" "47k"
+		(property "Value" "100k"
 			(at 249.936 85.09 0)
 			(effects
