File: Robot WallA/Robot WallA.kicad_pcb (KiCad board)
At the start: 2 copper layers, 263 parts, among them IC1 STM32F407IGT6, IC2 DS04-254-2-04BK-SMT, IC3 USBLC6-4SC6, IC4 USBLC6-4SC6, IC5 LAN8742A-CZ-TR, IC6 TLV75533PDBVR, IC7 ABXS005A4X341-SRZ, IC8 DRV8262DDVR, IC9 74LVC2G241DP-Q100H, J1 NC-Conn_02x05_Female, J10 Conn_01x02, J11 NID35-5, J12 NID35-5, J13 39501-1002, J14 39501-1002, J15 39501-1004, J16 39501-1004, J17 22-03-5035, J18 22-03-5035, J19 22-03-5035, J2 USB4216-03-A, J20 22-03-5035, J21 Conn_01x03, J22 281695-3, J23 Conn_01x03, J24 281695-3, J25 Conn_01x03, J26 281695-3, J27 Conn_01x03, J28 39501-1002, J29 39501-1002, J3 SS-90000-009, J30 Conn_01x03, J31 281695-3, J4 USB_B_Micro, J5 Conn_02x36_Counter_Clockwise, J6 Conn_02x36_Counter_Clockwise, J7 Conn_01x02, J8 XT90PW_M, J9 Conn_01x02, Q1 BSS138, Q2 BSS138, Q3 BSS138, Q4 BSS119, Q5 BSS119, SW1 Switch, T1 H1102NL, U1 FT230XS, U2 125700D00000G, U3 125700D00000G, U4 125700D00000G, U5 125700D00000G, U6 L298N, Y1 Crystal_GND24

Commit message: Added standard switchs, debug leds and 12V and 5V connectors
Parts:
- removed D16: LED_RED, LED_SMD:LED_0603_1608Metric
- removed R53: 1.6k, Resistor_SMD:R_0603_1608Metric_Pad0.98x0.95mm_HandSolder
- added D14: 1N5819, Diode_SMD:D_SOD-123, F.Cu at (-56.3, 146.9)
- added D17: LED, LED_SMD:LED_0603_1608Metric, F.Cu at (166.2, 242.0)
- added D18: LED, LED_SMD:LED_0603_1608Metric, F.Cu at (166.2, 244.6)
- added D19: LED, LED_SMD:LED_0603_1608Metric, F.Cu at (166.2, 247.2)
- added D20: LED, LED_SMD:LED_0603_1608Metric, F.Cu at (166.2, 249.8)
- added D21: LED, LED_SMD:LED_0603_1608Metric, F.Cu at (166.2, 252.3)
- added J32: Conn_01x03, Connector_PinHeader_2.54mm:PinHeader_1x03_P2.54mm_Vertical, F.Cu at (-76.7, 153.2)
- added J33: 281695-3, SamacSys_Parts:SHDR3W65P0X254_1X3_762X508X1150P, F.Cu at (-66.4, 148.3)
- added J34: Conn_01x03, Connector_PinHeader_2.54mm:PinHeader_1x03_P2.54mm_Vertical, F.Cu at (238.5, 84.4)
- added J35: BM04B-SRSS-TB, SamacSys_Parts:BM04B-SRSS-TB_LFSN_, F.Cu at (240.9, 92.5)
- added J36: BM04B-SRSS-TB, SamacSys_Parts:BM04B-SRSS-TB_LFSN_, F.Cu at (249.6, 92.5)
- added J37: BM04B-SRSS-TB, SamacSys_Parts:BM04B-SRSS-TB_LFSN_, F.Cu at (258.3, 92.5)
- added J38: BM02B-SRSS-TB, SamacSys_Parts:BM02BSRSSTBLFSN, F.Cu at (267.0, 92.5)
- added J39: Conn_01x03, Connector_PinHeader_2.54mm:PinHeader_1x03_P2.54mm_Vertical, F.Cu at (238.5, 79.8)
- added J40: BM03B-SRSS-TB, SamacSys_Parts:BM03BSRSSTB, F.Cu at (250.0, 82.3)
- added J41: BM03B-SRSS-TB, SamacSys_Parts:BM03BSRSSTB, F.Cu at (257.3, 82.3)
- added J42: BM03B-SRSS-TB, SamacSys_Parts:BM03BSRSSTB, F.Cu at (264.6, 82.3)
- added J43: BM03B-SRSS-TB, SamacSys_Parts:BM03BSRSSTB, F.Cu at (271.9, 82.3)
- added J44: BM02B-SRSS-TB, SamacSys_Parts:BM02BSRSSTBLFSN, F.Cu at (251.3, 101.7)
- added J45: BM04B-SRSS-TB, SamacSys_Parts:BM04B-SRSS-TB_LFSN_, F.Cu at (240.9, 101.1)
- added J46: BM02B-SRSS-TB, SamacSys_Parts:BM02BSRSSTBLFSN, F.Cu at (258.9, 101.7)
- added J47: BM02B-SRSS-TB, SamacSys_Parts:BM02BSRSSTBLFSN, F.Cu at (266.4, 101.7)
- added R51: 0.5R/0.1%, Resistor_SMD:R_0603_1608Metric_Pad0.98x0.95mm_HandSolder, F.Cu at (-42.6, 148.9)
- added R55: 649R, Resistor_SMD:R_0603_1608Metric, F.Cu at (170.2, 241.9)
- added R56: 750R, Resistor_SMD:R_0603_1608Metric, F.Cu at (170.2, 244.5)
- added R57: 324R, Resistor_SMD:R_0603_1608Metric, F.Cu at (170.2, 247.0)
- added R58: 330R, Resistor_SMD:R_0603_1608Metric, F.Cu at (170.2, 249.5)
- added R59: 549R, Resistor_SMD:R_0603_1608Metric, F.Cu at (170.2, 252.0)
- added TP3: 24V, TestPoint:TestPoint_Pad_D2.0mm, F.Cu at (15.6, -95.2)
- added TP4: 12V, TestPoint:TestPoint_Pad_D2.0mm, F.Cu at (15.6, -91.1)
- added TP5: 5V_COMPUTE, TestPoint:TestPoint_Pad_D2.0mm, F.Cu at (15.6, -87.0)
- added TP6: 5V_ACTUATORS, TestPoint:TestPoint_Pad_D2.0mm, F.Cu at (15.6, -83.0)
- added TP7: 3V3, TestPoint:TestPoint_Pad_D2.0mm, F.Cu at (15.6, -79.0)
- D13, D15: value LED_RED -> 1N5819; footprint LED_SMD:LED_0603_1608Metric -> Diode_SMD:D_SOD-123
- D5, D6, D7: value 1N5819 -> LED_RED; footprint Diode_SMD:D_SOD-123 -> LED_SMD:LED_0603_1608Metric
- J1: value NC-Conn_02x05_Female -> Conn_02x05_Female
- J10, J9: footprint Connector_PinHeader_2.54mm:PinHeader_1x02_P2.54mm_Vertical -> SamacSys_Parts:SHDR2W50P0X200_1X2_590X450X600P
- J11, J12: value NID35-5 -> Conn_01x02; footprint SamacSys_Parts:NID355 -> Connector_PinHeader_2.54mm:PinHeader_1x02_P2.54mm_Vertical
- J13, J14: value 39501-1002 -> NID35-5; footprint SamacSys_Parts:395011002 -> SamacSys_Parts:NID355
- J15, J16: value 39501-1004 -> 39501-1002; footprint SamacSys_Parts:395011004 -> SamacSys_Parts:395011002
- J17, J18: value 22-03-5035 -> 39501-1004; footprint SamacSys_Parts:SHDR3W60P0X250_1X3_990X490X590P -> SamacSys_Parts:395011004
- J21: value Conn_01x03 -> 22-03-5035; footprint Connector_PinHeader_2.54mm:PinHeader_1x03_P2.54mm_Vertical -> SamacSys_Parts:SHDR3W60P0X250_1X3_990X490X590P
- J22: value 281695-3 -> 22-03-5035; footprint SamacSys_Parts:SHDR3W65P0X254_1X3_762X508X1150P -> SamacSys_Parts:SHDR3W60P0X250_1X3_990X490X590P
- J28: value 39501-1002 -> 281695-3; footprint SamacSys_Parts:395011002 -> SamacSys_Parts:SHDR3W65P0X254_1X3_762X508X1150P
- J29: value 39501-1002 -> Conn_01x03; footprint SamacSys_Parts:395011002 -> Connector_PinHeader_2.54mm:PinHeader_1x03_P2.54mm_Vertical
- J30: value Conn_01x03 -> 39501-1002; footprint Connector_PinHeader_2.54mm:PinHeader_1x03_P2.54mm_Vertical -> SamacSys_Parts:395011002
- J31: value 281695-3 -> 39501-1002; footprint SamacSys_Parts:SHDR3W65P0X254_1X3_762X508X1150P -> SamacSys_Parts:395011002
- R30: value 100k -> 1.6k
- R31, R40, R46: value 10k -> 100k
- R32: value 200k -> 10k
- R33: value 100k -> 11.1k
- R34: value 10k -> 200k
- R35: value 10,553k/1% -> 100k
- R37: value 100k -> 10,553k/1%
- R39: value 10k -> 5.1k
- R41, R42: value 3,09k -> 10k
- R43: value 100k -> 10k
- R44, R45: value 10k -> 3,09k
- R48, R49: value 0.5R/0.1% -> 10k
- R50: value 11.1k -> 10k
- R52: value 5.1k -> 0.5R/0.1%
- U1: value FT230XS -> FT231XS; footprint Package_SO:SSOP-16_3.9x4.9mm_P0.635mm -> Package_SO:SSOP-20_3.9x8.7mm_P0.635mm
- moved J18 445.0 mm to (245.3, 66.1)
- moved J17 444.7 mm to (245.3, 56.1)
- moved C13 362.0 mm to (141.9, 263.1)
- moved C14 362.0 mm to (141.9, 265.6)
- moved C21 362.0 mm to (146.3, 263.1)
- moved C22 362.0 mm to (146.3, 265.6)
- moved C5 362.0 mm to (137.6, 263.1)
- moved C6 362.0 mm to (137.6, 265.6)
- moved JP1 362.0 mm to (151.3, 258.6)
- moved C10 362.0 mm to (137.6, 275.6)
- moved C11 362.0 mm to (141.9, 258.1)
- moved C12 362.0 mm to (141.9, 260.6)
- moved C15 362.0 mm to (141.9, 268.1)
- moved C16 362.0 mm to (141.9, 270.6)
- moved C17 362.0 mm to (141.9, 273.1)
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Connections:
- D10 pad 1: Net-(D10-K) -> /Motor/Motor_Actuators/PWR_5
- D10 pad 2: GND -> Net-(D10-A)
- D11 pad 1: Net-(D11-K) -> /Motor/Motor_Actuators/PWR_5
- D11 pad 2: GND -> Net-(D11-A)
- D13 pad 2: /Power/24V -> GND
- D15 pad 1: Net-(D15-K) -> Net-(D11-A)
- D15 pad 2: /Power/12V -> GND
- D5 pad 1: /Motor/Motor_Actuators/PWR_5 -> Net-(D5-K)
- D5 pad 2: Net-(D5-A) -> /Motor/5V
- D6 pad 1: /Motor/Motor_Actuators/PWR_5 -> Net-(D6-K)
- D6 pad 2: Net-(D10-K) -> /Power/24V
- D7 pad 1: /Motor/Motor_Actuators/PWR_5 -> Net-(D7-K)
- D7 pad 2: Net-(D11-K) -> /Power/12V
- D9 pad 1: Net-(D5-A) -> /Motor/Motor_Actuators/PWR_5
- D9 pad 2: GND -> Net-(D13-K)
- F3 pad 1: Net-(J9-Pin_2) -> Net-(J11-Pin_2)
- F4 pad 1: Net-(J10-Pin_2) -> Net-(J12-Pin_2)
- IC1 pad 115: /MCU/ENCODER0 -> /MCU/SENSORS11
- IC1 pad 116: /MCU/ENCODER1 -> /MCU/SENSORS10
- IC1 pad 117: /MCU/MCU_Core/PC8 -> /MCU/SENSORS9
- IC1 pad 118: /MCU/MCU_Core/PC9 -> /MCU/SENSORS8
- IC1 pad 162: /MCU/MCU_Core/PB4 -> /MCU/ENCODER0
- IC1 pad 163: /MCU/MCU_Core/PB5 -> /MCU/ENCODER1
- IC1 pad 32: /MCU/MCU_Core/PC0 -> /MCU/SENSORS1
- IC1 pad 34: /MCU/MCU_Core/PC2 -> /MCU/SENSORS2
- IC1 pad 35: /MCU/MCU_Core/PC3 -> /MCU/SENSORS3
- IC1 pad 57: /MCU/MCU_Core/PB1 -> /MCU/SENSORS0
- J10 pad 1: /Power/Vbatt -> GND
- J10 pad 2: Net-(J10-Pin_2) -> /Motor/5V
- J11 pad 1: /MCU/5V_PC_EMBARQUE -> /Power/Vbatt
- J11 pad 2: /MCU/5V_PC_EMBARQUE -> Net-(J11-Pin_2)
- J12 pad 1: /Motor/5V -> /Power/Vbatt
- J12 pad 2: /Motor/5V -> Net-(J12-Pin_2)
- J13 pad 1: /Motor/Motor_WheelDriver/Motor1_High -> /MCU/5V_PC_EMBARQUE
- J13 pad 2: /Motor/Motor_WheelDriver/Motor1_Low -> /MCU/5V_PC_EMBARQUE
- J14 pad 1: /Motor/Motor_WheelDriver/Motor2_High -> /Motor/5V
- J14 pad 2: /Motor/Motor_WheelDriver/Motor2_Low -> /Motor/5V
- J15 pad 1: /Motor/5V -> /Motor/Motor_WheelDriver/Motor1_High
- J15 pad 2: /MCU/ENCODER0 -> /Motor/Motor_WheelDriver/Motor1_Low
- J16 pad 1: /Motor/5V -> /Motor/Motor_WheelDriver/Motor2_High
- J16 pad 2: /MCU/ENCODER2 -> /Motor/Motor_WheelDriver/Motor2_Low
- J17 pad 1: /Motor/Motor_Actuators/DATA -> /Motor/5V
- J17 pad 2: /Power/12V -> /MCU/ENCODER0
- J17 pad 3: GND -> /MCU/ENCODER1
- J18 pad 1: /Motor/Motor_Actuators/DATA -> /Motor/5V
- J18 pad 2: /Power/12V -> /MCU/ENCODER2
- J18 pad 3: GND -> /MCU/ENCODER3
- J21 pad 1: /Power/12V -> /Motor/Motor_Actuators/DATA
- J21 pad 2: /Motor/Motor_Actuators/PWR_5 -> /Power/12V
- J21 pad 3: /Motor/5V -> GND
- J22 pad 1: GND -> /Motor/Motor_Actuators/DATA
- J22 pad 2: /Motor/Motor_Actuators/PWR_1 -> /Power/12V
- J22 pad 3: /MCU/SERVO3 -> GND
- J23 pad 2: /Motor/Motor_Actuators/PWR_1 -> /Motor/Motor_Actuators/PWR_5
- J24 pad 2: /Motor/Motor_Actuators/PWR_2 -> /Motor/Motor_Actuators/PWR_1
- J24 pad 3: /MCU/SERVO4 -> /MCU/SERVO3
- J25 pad 2: /Motor/Motor_Actuators/PWR_2 -> /Motor/Motor_Actuators/PWR_1
- J26 pad 2: /Motor/Motor_Actuators/PWR_3 -> /Motor/Motor_Actuators/PWR_2
- J26 pad 3: /MCU/SERVO5 -> /MCU/SERVO4
- J27 pad 2: /Motor/Motor_Actuators/PWR_3 -> /Motor/Motor_Actuators/PWR_2
- J28 pad 1: Net-(D5-A) -> GND
- J28 pad 2: Net-(D10-K) -> /Motor/Motor_Actuators/PWR_3
- J29 pad 1: Net-(D11-K) -> /Power/12V
- J29 pad 2: Net-(D12-K) -> /Motor/Motor_Actuators/PWR_3
- J30 pad 1: /Power/12V -> Net-(D12-K)
- J30 pad 2: /Motor/Motor_Actuators/PWR_4 -> Net-(D13-K)
- J31 pad 1: GND -> Net-(D10-A)
- J31 pad 2: /Motor/Motor_Actuators/PWR_4 -> Net-(D11-A)
- J9 pad 1: /Power/Vbatt -> GND
- J9 pad 2: Net-(J9-Pin_2) -> /Power/12V
- R30 pad 1: /Motor/5V -> Net-(D5-K)
- R30 pad 2: /Power/Power_Buck_5V_Actuators/ENABLE -> GND
- R31 pad 1: /Power/GPIO_ENABLE_POWER_SUPPLIES -> /Motor/5V
- R31 pad 2: GND -> /Power/Power_Buck_5V_Actuators/ENABLE
- R32 pad 1: Net-(C82-Pad2) -> /Power/GPIO_ENABLE_POWER_SUPPLIES
- R32 pad 2: /Power/Power_Boost_24V/SENSE+ -> GND
- R33 pad 1: /Power/Power_Boost_24V/IN -> Net-(D6-K)
- R33 pad 2: /Power/Power_Boost_24V/ENABLE -> GND
- R34 pad 1: /Power/GPIO_PGOOD -> Net-(C82-Pad2)
- R34 pad 2: /MCU/3V3 -> /Power/Power_Boost_24V/SENSE+
- R35 pad 1: GND -> /Power/Power_Boost_24V/IN
- R35 pad 2: /Power/Power_Boost_24V/TRIM -> /Power/Power_Boost_24V/ENABLE
- R36 pad 1: /Power/GPIO_ENABLE_POWER_SUPPLIES -> /Power/GPIO_PGOOD
- R36 pad 2: GND -> /MCU/3V3
- R37 pad 1: /Power/12V -> GND
- R37 pad 2: /Power/Power_Buck_12V/ENABLE -> /Power/Power_Boost_24V/TRIM
- R39 pad 1: /MCU/WHEEL6 -> Net-(D7-K)
- R39 pad 2: /MCU/3V3 -> GND
- R40 pad 1: Net-(IC8-OCPM) -> /Power/12V
- R40 pad 2: /MCU/3V3 -> /Power/Power_Buck_12V/ENABLE
- R41 pad 1: GND -> /Power/GPIO_ENABLE_POWER_SUPPLIES
- R41 pad 2: /MCU/WHEEL0 -> GND
- R42 pad 1: GND -> /MCU/WHEEL6
- R42 pad 2: /MCU/WHEEL1 -> /MCU/3V3
- R43 pad 1: GND -> Net-(IC8-OCPM)
- R43 pad 2: /Motor/Motor_WheelDriver/TOFF -> /MCU/3V3
- R44 pad 1: /Motor/5V -> GND
- R44 pad 2: /Motor/Motor_Actuators/TX_UC_5V -> /MCU/WHEEL0
- R45 pad 1: /MCU/SERVO2 -> GND
- R45 pad 2: GND -> /MCU/WHEEL1
- R46 pad 1: /Motor/5V -> GND
- R46 pad 2: /Motor/Motor_Actuators/RX_UC_5V -> /Motor/Motor_WheelDriver/TOFF
- R47 pad 2: /Motor/Motor_Actuators/DATA -> /Motor/Motor_Actuators/TX_UC_5V
- R48 pad 1: Net-(JP9-B) -> /MCU/SERVO2
- R49 pad 1: Net-(JP10-B) -> /Motor/5V
- R49 pad 2: GND -> /Motor/Motor_Actuators/RX_UC_5V
- R50 pad 1: Net-(D13-K) -> /Motor/5V
- R50 pad 2: GND -> /Motor/Motor_Actuators/DATA
- R52 pad 1: Net-(D15-K) -> Net-(JP10-B)
- RV1 pad 2: Net-(J11-TRIM(OPTIONAL)) -> Net-(J13-TRIM(OPTIONAL))
- RV2 pad 2: Net-(J12-TRIM(OPTIONAL)) -> Net-(J14-TRIM(OPTIONAL))
- U1 pad 1: /MCU/MCU_Core/PA10 -> unconnected-(U1-~{DTR}-Pad1)
- U1 pad 10: /MCU/MCU_Debug/3V3 -> Net-(U1-CBUS2)
- U1 pad 11: /MCU/MCU_Core/NRST -> Net-(J4-D+)
- U1 pad 12: /MCU/MCU_Debug/5V_DEBUG -> Net-(J4-D-)
- U1 pad 13: GND -> /MCU/MCU_Debug/3V3
- U1 pad 14: Net-(U1-CBUS1) -> /MCU/MCU_Core/NRST
- U1 pad 15: unconnected-(U1-CBUS0-Pad15) -> /MCU/MCU_Debug/5V_DEBUG
- U1 pad 16: unconnected-(U1-CBUS3-Pad16) -> GND
- U1 pad 5: GND -> unconnected-(U1-~{RI}-Pad5)
- U1 pad 6: unconnected-(U1-~{CTS}-Pad6) -> GND
- U1 pad 7: Net-(U1-CBUS2) -> unconnected-(U1-~{DSR}-Pad7)
- U1 pad 8: Net-(J4-D+) -> unconnected-(U1-~{DCD}-Pad8)
- U1 pad 9: Net-(J4-D-) -> unconnected-(U1-~{CTS}-Pad9)
- U6 pad 13: Net-(D11-K) -> Net-(D10-A)
- U6 pad 14: Net-(D12-K) -> Net-(D11-A)
- U6 pad 2: Net-(D5-A) -> Net-(D12-K)
- U6 pad 3: Net-(D10-K) -> Net-(D13-K)
Other:
- board outline added: 170 x 100 mm
- copper layers 2 -> 4

Commit message: Begin to route ethenet, usb, 24V power supply.
Reworked Ethernet sheet because it was too hard to read
Parts:
- removed IC5: LAN8742A-CZ-TR, SamacSys_Parts:QFN50P400X400X100-25N-D
- removed J5: Conn_02x36_Counter_Clockwise, Connector_PinHeader_2.54mm:PinHeader_2x36_P2.54mm_Vertical
- removed R26: 10K, Resistor_SMD:R_0603_1608Metric_Pad0.98x0.95mm_HandSolder
- added C115: 470pF, Capacitor_SMD:C_0603_1608Metric_Pad1.08x0.95mm_HandSolder, F.Cu at (39.7, 225.0)
- added C116: 100nF, Capacitor_SMD:C_0603_1608Metric_Pad1.08x0.95mm_HandSolder, F.Cu at (54.2, 232.4)
- added JP11: Open, Jumper:SolderJumper-2_P1.3mm_Open_RoundedPad1.0x1.5mm, F.Cu at (59.1, 219.8)
- added U7: LAN8742A, Package_DFN_QFN:VQFN-24-1EP_4x4mm_P0.5mm_EP2.5x2.5mm_ThermalVias, F.Cu at (44.1, 228.6)
- added Y2: Crystal_GND24, Crystal:Crystal_SMD_3225-4Pin_3.2x2.5mm, F.Cu at (43.4, 222.1)
- C23: value 100nF -> 10uF; footprint Capacitor_SMD:C_0603_1608Metric_Pad1.08x0.95mm_HandSolder -> Capacitor_SMD:C_1206_3216Metric_Pad1.33x1.80mm_HandSolder
- C24: value 10uF -> 100nF
- C27, C28: value 100nF -> 12pF
- C29: value 1nF -> 100nF
- C30: value 470pF -> 100nF
- C31: value 1uF -> 1nF; footprint Capacitor_SMD:C_0603_1608Metric_Pad1.08x0.95mm_HandSolder -> Capacitor_SMD:C_1206_3216Metric_Pad1.33x1.80mm_HandSolder
- C32: value 100nF -> 1uF
- FB2: value Bead 600R -> FerriteBead
- JP4: value SolderJumper -> Closed; footprint Jumper:SolderJumper-2_P1.3mm_Open_Pad1.0x1.5mm -> Jumper:SolderJumper-2_P1.3mm_Bridged_RoundedPad1.0x1.5mm
- JP5: value SolderJumper -> Open; footprint Jumper:SolderJumper-2_P1.3mm_Open_Pad1.0x1.5mm -> Jumper:SolderJumper-2_P1.3mm_Open_RoundedPad1.0x1.5mm
- R10, R9: value 75R -> 10k; footprint Resistor_SMD:R_0603_1608Metric_Pad0.98x0.95mm_HandSolder -> Resistor_SMD:R_0603_1608Metric
- R11, R12: value 75R -> 33R; footprint Resistor_SMD:R_0603_1608Metric_Pad0.98x0.95mm_HandSolder -> Resistor_SMD:R_0603_1608Metric
- R13: value 0R -> 10k; footprint Resistor_SMD:R_0603_1608Metric_Pad0.98x0.95mm_HandSolder -> Resistor_SMD:R_0603_1608Metric
- R14, R18, R4, R5, R6, R7: footprint Resistor_SMD:R_0603_1608Metric_Pad0.98x0.95mm_HandSolder -> Resistor_SMD:R_0603_1608Metric
- R15, R17: value 270R -> 1k5; footprint Resistor_SMD:R_0603_1608Metric_Pad0.98x0.95mm_HandSolder -> Resistor_SMD:R_0603_1608Metric
- R16: value 10K -> 12k1; footprint Resistor_SMD:R_0603_1608Metric_Pad0.98x0.95mm_HandSolder -> Resistor_SMD:R_0603_1608Metric
- R19: value 10K -> 270R; footprint Resistor_SMD:R_0603_1608Metric_Pad0.98x0.95mm_HandSolder -> Resistor_SMD:R_0603_1608Metric
- R20: value 10K -> 10k; footprint Resistor_SMD:R_0603_1608Metric_Pad0.98x0.95mm_HandSolder -> Resistor_SMD:R_0603_1608Metric
- R21: value 33R -> 270R; footprint Resistor_SMD:R_0603_1608Metric_Pad0.98x0.95mm_HandSolder -> Resistor_SMD:R_0603_1608Metric
- R22: value 1.5k -> 75R; footprint Resistor_SMD:R_0603_1608Metric_Pad0.98x0.95mm_HandSolder -> Resistor_SMD:R_0603_1608Metric
- R23, R24: value 10K -> 75R; footprint Resistor_SMD:R_0603_1608Metric_Pad0.98x0.95mm_HandSolder -> Resistor_SMD:R_0603_1608Metric
- R25: value 33R -> 75R; footprint Resistor_SMD:R_0603_1608Metric_Pad0.98x0.95mm_HandSolder -> Resistor_SMD:R_0603_1608Metric
- R8: value 12.1k -> 10k; footprint Resistor_SMD:R_0603_1608Metric_Pad0.98x0.95mm_HandSolder -> Resistor_SMD:R_0603_1608Metric
- moved U2 251.8 mm to (117.8, 92.5), turned to -90 degrees
- moved TP3 202.5 mm to (96.0, 90.8), turned to 180 degrees
- moved IC7 193.8 mm to (100.0, 68.3), turned to 180 degrees
- moved C62 186.5 mm to (83.5, 98.8), turned to 180 degrees
- moved Q2 169.2 mm to (117.0, 77.4), turned to 90 degrees
- moved D6 164.7 mm to (97.5, 95.8), turned to 180 degrees
- moved C63 159.7 mm to (98.5, 87.8)
- moved R33 155.9 mm to (97.5, 97.6), turned to 180 degrees
- moved C64 154.4 mm to (93.8, 87.8), turned to 180 degrees
- moved R36 154.2 mm to (111.5, 83.1), turned to 180 degrees
- moved R35 152.0 mm to (116.2, 73.5), turned to -90 degrees
- moved R38 151.9 mm to (117.0, 80.2)
- moved C65 151.6 mm to (98.5, 83.2)
- moved C66 151.0 mm to (98.5, 85.5)
- moved TP5 149.7 mm to (162.5, -58.0)
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Connections:
- net Net-(T1-RX+) renamed /MCU/MCU_Peripherals/RX+
- net Net-(T1-RX-) renamed /MCU/MCU_Peripherals/RX-
- net Net-(T1-TX+) renamed /MCU/MCU_Peripherals/TX+
- net Net-(T1-TX-) renamed /MCU/MCU_Peripherals/TX-
- C23 pad 1: Net-(C24-+) -> /MCU/MCU_Peripherals/3V3_filtered
- C24 pad 1: Net-(C24-+) -> /MCU/MCU_Peripherals/3V3_filtered
- C25 pad 1: Net-(C24-+) -> /MCU/MCU_Peripherals/3V3_filtered
- C26 pad 1: GND -> /MCU/MCU_Peripherals/3V3
- C26 pad 2: Net-(C24-+) -> GND
- C27 pad 1: GND -> /MCU/MCU_Peripherals/Q+
- C27 pad 2: Net-(C24-+) -> GND
- C28 pad 1: GND -> /MCU/MCU_Peripherals/Q-
- C28 pad 2: Net-(C24-+) -> GND
- C29 pad 1: GNDPWR -> /MCU/MCU_Peripherals/3V3_filtered
- C29 pad 2: Net-(C29-Pad2) -> GND
- C30 pad 1: Net-(IC5-VDDCR) -> /MCU/MCU_Peripherals/3V3_filtered
- C31 pad 1: Net-(IC5-VDDCR) -> Net-(C31-Pad1)
- C31 pad 2: GND -> GNDPWR
- C32 pad 1: GND -> /MCU/MCU_Peripherals/VDDCR
- C32 pad 2: /MCU/3V3 -> GND
- FB2 pad 1: /MCU/3V3 -> /MCU/MCU_Peripherals/3V3
- FB2 pad 2: Net-(C24-+) -> /MCU/MCU_Peripherals/3V3_filtered
- IC3 pad 4: /MCU/MCU_Peripherals/CC1 -> /MCU/MCU_Peripherals/CC2
- IC3 pad 6: /MCU/MCU_Peripherals/CC2 -> /MCU/MCU_Peripherals/CC1
- IC4 pad 1: Net-(IC4-I/O1) -> /MCU/MCU_Peripherals/RXN
- IC4 pad 3: Net-(IC4-I/O2) -> /MCU/MCU_Peripherals/RXP
- IC4 pad 4: Net-(IC4-I/O3) -> /MCU/MCU_Peripherals/TXP
- IC4 pad 5: Net-(C24-+) -> /MCU/MCU_Peripherals/3V3_filtered
- IC4 pad 6: Net-(IC4-I/O4) -> /MCU/MCU_Peripherals/TXN
- J3 pad 10: Net-(IC5-LED2/NINT/NPME/NINTSEL) -> /MCU/MCU_Peripherals/LED_Green
- J3 pad 12: Net-(C24-+) -> /MCU/MCU_Peripherals/LED_Yellow
- J3 pad 4: Net-(T1-NC_6) -> Net-(J3-Pad4)
- J3 pad 5: Net-(T1-NC_6) -> Net-(J3-Pad4)
- J6 pad 1: /MCU/3V3 -> unconnected-(J6-Pin_1-Pad1)
- J6 pad 10: /MCU/MCU_Core/PA0 -> unconnected-(J6-Pin_10-Pad10)
- J6 pad 11: /MCU/MCU_Core/PA2 -> unconnected-(J6-Pin_11-Pad11)
- J6 pad 12: /MCU/MCU_Core/PA8 -> unconnected-(J6-Pin_12-Pad12)
- J6 pad 13: /MCU/MCU_Core/PB1 -> unconnected-(J6-Pin_13-Pad13)
- J6 pad 14: /MCU/MCU_Core/PC7 -> unconnected-(J6-Pin_14-Pad14)
- J6 pad 15: /MCU/MCU_Core/PC9 -> unconnected-(J6-Pin_15-Pad15)
- J6 pad 16: /MCU/MCU_Core/PA13 -> unconnected-(J6-Pin_16-Pad16)
- J6 pad 17: /MCU/MCU_GPIO/NRST -> unconnected-(J6-Pin_17-Pad17)
- J6 pad 18: /MCU/MCU_Core/PC0 -> unconnected-(J6-Pin_18-Pad18)
- J6 pad 19: /MCU/MCU_Core/PC2 -> unconnected-(J6-Pin_19-Pad19)
- J6 pad 2: /MCU/MCU_Core/PA9 -> unconnected-(J6-Pin_2-Pad2)
- J6 pad 20: /MCU/MCU_Core/PC4 -> unconnected-(J6-Pin_20-Pad20)
- J6 pad 21: /MCU/MCU_Core/PC11 -> unconnected-(J6-Pin_21-Pad21)
- J6 pad 22: /MCU/MCU_Core/PD0 -> unconnected-(J6-Pin_22-Pad22)
- J6 pad 23: /MCU/MCU_Core/PD2 -> unconnected-(J6-Pin_23-Pad23)
- J6 pad 24: /MCU/MCU_Core/PD4 -> unconnected-(J6-Pin_24-Pad24)
- J6 pad 25: /MCU/MCU_Core/PD6 -> unconnected-(J6-Pin_25-Pad25)
- J6 pad 26: /MCU/MCU_Core/PD8 -> unconnected-(J6-Pin_26-Pad26)
- J6 pad 27: /MCU/MCU_Core/PD10 -> unconnected-(J6-Pin_27-Pad27)
- J6 pad 28: /MCU/MCU_Core/PD12 -> unconnected-(J6-Pin_28-Pad28)
- J6 pad 29: /MCU/MCU_Core/PD14 -> unconnected-(J6-Pin_29-Pad29)
- J6 pad 3: /MCU/MCU_Core/PA2 -> unconnected-(J6-Pin_3-Pad3)
- J6 pad 30: /MCU/MCU_Core/PE0 -> unconnected-(J6-Pin_30-Pad30)
- J6 pad 31: /MCU/MCU_Core/PE2 -> unconnected-(J6-Pin_31-Pad31)
- J6 pad 32: /MCU/MCU_Core/PE4 -> unconnected-(J6-Pin_32-Pad32)
- J6 pad 33: /MCU/MCU_Core/PE6 -> unconnected-(J6-Pin_33-Pad33)
- J6 pad 34: /MCU/MCU_Core/PE8 -> unconnected-(J6-Pin_34-Pad34)
- J6 pad 35: /MCU/MCU_Core/PE10 -> unconnected-(J6-Pin_35-Pad35)
- J6 pad 36: /MCU/5V_PC_EMBARQUE -> unconnected-(J6-Pin_36-Pad36)
- J6 pad 37: GND -> unconnected-(J6-Pin_37-Pad37)
- J6 pad 38: /MCU/MCU_Core/PE11 -> unconnected-(J6-Pin_38-Pad38)
- J6 pad 39: /MCU/MCU_Core/PE9 -> unconnected-(J6-Pin_39-Pad39)
- J6 pad 4: /MCU/MCU_Core/PB6 -> unconnected-(J6-Pin_4-Pad4)
- J6 pad 40: /MCU/MCU_Core/PE7 -> unconnected-(J6-Pin_40-Pad40)
- J6 pad 41: /MCU/MCU_Core/PE5 -> unconnected-(J6-Pin_41-Pad41)
- J6 pad 42: /MCU/MCU_Core/PE3 -> unconnected-(J6-Pin_42-Pad42)
- J6 pad 43: /MCU/MCU_Core/PE1 -> unconnected-(J6-Pin_43-Pad43)
- J6 pad 44: /MCU/MCU_Core/PD15 -> unconnected-(J6-Pin_44-Pad44)
- J6 pad 45: /MCU/MCU_Core/PD13 -> unconnected-(J6-Pin_45-Pad45)
- J6 pad 46: /MCU/MCU_Core/PD11 -> unconnected-(J6-Pin_46-Pad46)
- J6 pad 47: /MCU/MCU_Core/PD9 -> unconnected-(J6-Pin_47-Pad47)
- J6 pad 48: /MCU/MCU_Core/PD7 -> unconnected-(J6-Pin_48-Pad48)
- J6 pad 49: /MCU/MCU_Core/PD5 -> unconnected-(J6-Pin_49-Pad49)
- J6 pad 5: /MCU/MCU_Core/PB10 -> unconnected-(J6-Pin_5-Pad5)
- J6 pad 50: /MCU/MCU_Core/PD3 -> unconnected-(J6-Pin_50-Pad50)
- J6 pad 51: /MCU/MCU_Core/PD1 -> unconnected-(J6-Pin_51-Pad51)
- J6 pad 52: /MCU/MCU_Core/PC12 -> unconnected-(J6-Pin_52-Pad52)
- J6 pad 53: /MCU/MCU_Core/PC5 -> unconnected-(J6-Pin_53-Pad53)
- J6 pad 54: /MCU/MCU_Core/PC3 -> unconnected-(J6-Pin_54-Pad54)
- J6 pad 55: /MCU/MCU_Core/PC1 -> unconnected-(J6-Pin_55-Pad55)
- J6 pad 56: /MCU/MCU_GPIO/BOOT0 -> unconnected-(J6-Pin_56-Pad56)
- J6 pad 57: /MCU/MCU_Core/PA14 -> unconnected-(J6-Pin_57-Pad57)
- J6 pad 58: /MCU/MCU_Core/PC10 -> unconnected-(J6-Pin_58-Pad58)
- J6 pad 59: /MCU/MCU_Core/PC8 -> unconnected-(J6-Pin_59-Pad59)
- J6 pad 6: /MCU/MCU_Core/PA5 -> unconnected-(J6-Pin_6-Pad6)
- J6 pad 60: /MCU/MCU_Core/PC6 -> unconnected-(J6-Pin_60-Pad60)
- J6 pad 61: /MCU/MCU_Core/PB0 -> unconnected-(J6-Pin_61-Pad61)
- J6 pad 62: /MCU/MCU_Core/PA3 -> unconnected-(J6-Pin_62-Pad62)
- J6 pad 63: /MCU/MCU_Core/PA1 -> unconnected-(J6-Pin_63-Pad63)
- J6 pad 64: /MCU/MCU_Core/PB12 -> unconnected-(J6-Pin_64-Pad64)
- J6 pad 65: /MCU/MCU_Core/PB14 -> unconnected-(J6-Pin_65-Pad65)
- J6 pad 66: /MCU/MCU_Core/PA4 -> unconnected-(J6-Pin_66-Pad66)
- J6 pad 67: /MCU/MCU_Core/PA6 -> unconnected-(J6-Pin_67-Pad67)
- J6 pad 68: /MCU/MCU_Core/PB11 -> unconnected-(J6-Pin_68-Pad68)
- J6 pad 69: /MCU/MCU_Core/PB7 -> unconnected-(J6-Pin_69-Pad69)
- J6 pad 7: /MCU/MCU_Core/PA7 -> unconnected-(J6-Pin_7-Pad7)
- J6 pad 70: /MCU/MCU_Core/PA3 -> unconnected-(J6-Pin_70-Pad70)
- J6 pad 71: /MCU/MCU_Core/PA10 -> unconnected-(J6-Pin_71-Pad71)
- J6 pad 8: /MCU/MCU_Core/PB13 -> unconnected-(J6-Pin_8-Pad8)
- J6 pad 9: /MCU/MCU_Core/PB15 -> unconnected-(J6-Pin_9-Pad9)
- JP4 pad 1: GNDPWR -> /MCU/MCU_Core/NRST
- JP4 pad 2: GND -> Net-(JP4-B)
- R10 pad 1: Net-(C29-Pad2) -> /MCU/MCU_Peripherals/3V3
- R10 pad 2: Net-(T1-NC_6) -> Net-(U7-CRS_DV/MODE2)
- R11 pad 1: Net-(C29-Pad2) -> /MCU/MCU_Core/ETH1
- R11 pad 2: Net-(T1-NC_6) -> Net-(U7-RXD0/MODE0)
- R12 pad 1: Net-(C29-Pad2) -> /MCU/MCU_Core/ETH2
- R12 pad 2: Net-(J3-Pad7) -> Net-(U7-RXD1/MODE1)
- R13 pad 1: Net-(IC5-NRST) -> GND
- R13 pad 2: /MCU/MCU_Core/NRST -> Net-(U7-RXER/PHYAD0)
- R14 pad 1: Net-(IC5-NINT/REFCLKO) -> /MCU/MCU_Core/ETH0
- R14 pad 2: /MCU/MCU_Core/ETH4 -> Net-(U7-CRS_DV/MODE2)
- R15 pad 1: GND -> /MCU/MCU_Peripherals/3V3
- R15 pad 2: Net-(J3-K_YELLOW) -> /MCU/MCU_Core/ETH5
- R16 pad 2: Net-(IC5-LED2/NINT/NPME/NINTSEL) -> Net-(U7-RBIAS)
- R17 pad 1: GND -> /MCU/MCU_Peripherals/3V3
- R17 pad 2: Net-(J3-K_GREEN) -> Net-(U7-~{INT}/REFCLKO)
- R18 pad 1: Net-(IC5-CRS_DV/MODE2) -> /MCU/MCU_Core/ETH4
- R18 pad 2: /MCU/MCU_Core/ETH0 -> Net-(U7-~{INT}/REFCLKO)
- R19 pad 1: /MCU/3V3 -> Net-(J3-K_YELLOW)
- R19 pad 2: Net-(IC5-RXD1/MODE1) -> GND
- R20 pad 1: /MCU/3V3 -> GND
- R20 pad 2: Net-(IC5-RXD0/MODE0) -> /MCU/MCU_Peripherals/LED_Green
- R21 pad 1: /MCU/MCU_Core/ETH2 -> Net-(J3-K_GREEN)
- R21 pad 2: Net-(IC5-RXD1/MODE1) -> GND
- R22 pad 1: /MCU/3V3 -> Net-(T1-NC_3)
- R22 pad 2: /MCU/MCU_Core/ETH3 -> Net-(C31-Pad1)
- R23 pad 1: /MCU/3V3 -> Net-(T1-NC_6)
- R23 pad 2: Net-(IC5-NINT/REFCLKO) -> Net-(C31-Pad1)
- R24 pad 1: /MCU/3V3 -> Net-(J3-Pad4)
- R24 pad 2: Net-(IC5-CRS_DV/MODE2) -> Net-(C31-Pad1)
- R25 pad 1: /MCU/MCU_Core/ETH1 -> Net-(J3-Pad7)
- R25 pad 2: Net-(IC5-RXD0/MODE0) -> Net-(C31-Pad1)
- R4 pad 1: Net-(IC4-I/O4) -> /MCU/MCU_Peripherals/3V3_filtered
- R4 pad 2: Net-(C24-+) -> /MCU/MCU_Peripherals/TXP
- R5 pad 1: Net-(IC4-I/O3) -> /MCU/MCU_Peripherals/3V3_filtered
- R5 pad 2: Net-(C24-+) -> /MCU/MCU_Peripherals/TXN
- R6 pad 1: Net-(IC4-I/O1) -> /MCU/MCU_Peripherals/3V3_filtered
- R6 pad 2: Net-(C24-+) -> /MCU/MCU_Peripherals/RXP
- R7 pad 1: Net-(IC4-I/O2) -> /MCU/MCU_Peripherals/3V3_filtered
- R7 pad 2: Net-(C24-+) -> /MCU/MCU_Peripherals/RXN
- R8 pad 1: Net-(IC5-RBIAS) -> /MCU/MCU_Peripherals/3V3
- R8 pad 2: GND -> Net-(U7-RXD0/MODE0)
- R9 pad 1: Net-(C29-Pad2) -> /MCU/MCU_Peripherals/3V3
- R9 pad 2: Net-(T1-NC_3) -> Net-(U7-RXD1/MODE1)
- T1 pad 1: Net-(IC4-I/O2) -> /MCU/MCU_Peripherals/RXP
- T1 pad 2: Net-(C24-+) -> /MCU/MCU_Peripherals/3V3_filtered
- T1 pad 3: Net-(IC4-I/O3) -> /MCU/MCU_Peripherals/RXN
- T1 pad 6: Net-(IC4-I/O1) -> /MCU/MCU_Peripherals/TXP
- T1 pad 7: Net-(C24-+) -> /MCU/MCU_Peripherals/3V3_filtered
- T1 pad 8: Net-(IC4-I/O4) -> /MCU/MCU_Peripherals/TXN
Routing:
- net /Power/Power_Boost_24V/IN: track 0.00 -> 30.6 mm
- net GNDPWR: track 0.00 -> 22.9 mm, vias 0 -> 3
- net Net-(C31-Pad1): track 0.00 -> 21.1 mm, vias 0 -> 2
- net Net-(J3-Pad4): track 0.00 -> 18.8 mm, vias 0 -> 1
- net /MCU/MCU_Peripherals/RXN: track 0.00 -> 18.4 mm
- net /MCU/MCU_Peripherals/RXP: track 0.00 -> 18.4 mm
- net /MCU/MCU_Peripherals/TXN: track 0.00 -> 17.9 mm
- net /MCU/MCU_Peripherals/TXP: track 0.00 -> 17.8 mm
- net Net-(J3-Pad7): track 0.00 -> 16.8 mm, vias 0 -> 1
- net /MCU/MCU_Peripherals/RX+: track 0.00 -> 13.5 mm
- net /MCU/MCU_Peripherals/RX-: track 0.00 -> 13.4 mm
- net /MCU/MCU_Peripherals/3V3_filtered: track 0.00 -> 12.2 mm, vias 0 -> 4
- net /MCU/MCU_Peripherals/TX+: track 0.00 -> 11.9 mm
- net /MCU/MCU_Peripherals/TX-: track 0.00 -> 11.8 mm
- net /MCU/5V_PC_EMBARQUE: track 0.00 -> 11.8 mm, vias 0 -> 1
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- added copper zone on F.Cu, net /Power/Power_Boost_24V/IN
- added copper zone on In2.Cu, net GNDPWR
- added copper zone on F.Cu, net Net-(J7-Pin_2)
Other:
- board text added: "12V"
- board text added: "24V"
- board text added: "3V3"
- board text added: "5V_ACTUATORS"
- board text added: "5V_COMPUTE"

Commit message: Continue to route
Parts:
- added C117: 120uF/25V, SamacSys_Parts:EEE0JA331XP, F.Cu at (65.8, 106.8)
- added C118: 47nF/25V, Capacitor_SMD:C_0603_1608Metric_Pad1.08x0.95mm_HandSolder, F.Cu at (79.2, 105.1)
- added C119: 47nF/25V, Capacitor_SMD:C_0603_1608Metric_Pad1.08x0.95mm_HandSolder, F.Cu at (83.7, 105.1)
- added C120: 47nF/25V, Capacitor_SMD:C_0603_1608Metric_Pad1.08x0.95mm_HandSolder, F.Cu at (59.7, 109.9)
- added C121: 4.7uF/25V, Capacitor_SMD:C_1210_3225Metric_Pad1.33x2.70mm_HandSolder, F.Cu at (78.6, 102.7)
- added C122: 4.7uF/25V, Capacitor_SMD:C_1210_3225Metric_Pad1.33x2.70mm_HandSolder, F.Cu at (84.3, 102.7)
- added C123: 22uF/25V, SamacSys_Parts:EEE1AA220WR, F.Cu at (126.4, 121.5)
- added C124: 4.7uF/50V, Capacitor_SMD:C_0805_2012Metric_Pad1.18x1.45mm_HandSolder, F.Cu at (113.2, 116.9)
- added C125: 4.7uF/50V, Capacitor_SMD:C_0805_2012Metric_Pad1.18x1.45mm_HandSolder, F.Cu at (115.8, 116.9)
- added C126: 4.7uF/50V, Capacitor_SMD:C_0805_2012Metric_Pad1.18x1.45mm_HandSolder, F.Cu at (118.3, 116.9)
- added C127: 10nF/50V, Capacitor_SMD:C_0805_2012Metric_Pad1.18x1.45mm_HandSolder, F.Cu at (120.8, 116.9)
- added C128: 100nF/50V, Capacitor_SMD:C_0603_1608Metric_Pad1.08x0.95mm_HandSolder, F.Cu at (189.6, 103.2)
- added C129: 100nF/50V, Capacitor_SMD:C_0603_1608Metric_Pad1.08x0.95mm_HandSolder, F.Cu at (189.6, 99.8)
- added R26: 0R, Resistor_SMD:R_0603_1608Metric_Pad0.98x0.95mm_HandSolder, F.Cu at (71.7, 170.3)
- C1, C10, C11, C12, C13, C14, C15, C16, C17, C18, C19, C2, C20, C21, C22, C3, C4, C5, C6, C7, C8, C9, FB1, IC1, J1, JP1, JP2, JP3, R1, SW1, Y1: moved to B.Cu
- C46, C57, C89: footprint Capacitor_SMD:C_0805_2012Metric_Pad1.18x1.45mm_HandSolder -> SamacSys_Parts:EEE1AA220WR
- C98, C99: value 100uF/50V -> 100nF/50V; footprint SamacSys_Parts:CAPAE830X1050N -> Capacitor_SMD:C_0603_1608Metric_Pad1.08x0.95mm_HandSolder
- TP1, TP2: footprint TestPoint:TestPoint_Pad_D2.0mm -> TestPoint:TestPoint_Pad_D1.0mm
- moved U4 333.9 mm to (201.4, 128.9), turned to -90 degrees
- moved J23 300.1 mm to (188.5, 54.9), turned to 90 degrees
- moved H5 291.4 mm to (203.9, 61.5)
- moved U6 291.4 mm to (182.3, 71.9)
- moved IC8 288.6 mm to (183.7, 104.8), turned to 180 degrees
- moved JP10 286.1 mm to (202.6, 76.8), turned to 180 degrees
- moved D11 281.2 mm to (216.0, 66.8), turned to 180 degrees
- moved C18 280.6 mm to (195.0, 0.15), turned to 180 degrees
- moved J30 280.2 mm to (220.9, 57.2), turned to 90 degrees
- moved J16 279.6 mm to (219.8, 108.4), turned to -90 degrees
- moved J15 279.4 mm to (219.8, 96.8), turned to -90 degrees
- moved D8 279.4 mm to (216.0, 64.4), turned to 180 degrees
- moved D10 279.3 mm to (216.0, 71.6), turned to 180 degrees
- moved D9 279.0 mm to (216.0, 69.2), turned to 180 degrees
- moved J31 277.2 mm to (221.0, 79.9), turned to 90 degrees
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Connections:
- net Net-(D10-A) renamed /Motor/Motor_Actuators/Motor2_High
- net Net-(D11-A) renamed /Motor/Motor_Actuators/Motor2_Low
- net Net-(D12-K) renamed /Motor/Motor_Actuators/Motor1_High
- net Net-(D13-K) renamed /Motor/Motor_Actuators/Motor1_Low
- net Net-(J4-D+) renamed /MCU/MCU_Debug/D+
- net Net-(J4-D-) renamed /MCU/MCU_Debug/D-
- C105 pad 1: /Motor/5V -> /Motor/Motor_Actuators/5V_ROBOTIS
- H5 pad 1: unconnected-(H5-Pad1) -> GND
- H5 pad 2: unconnected-(H5-Pad2) -> GND
- IC9 pad 8: /Motor/5V -> /Motor/Motor_Actuators/5V_ROBOTIS
- JP7 pad 1: /MCU/3V3 -> GND
- JP7 pad 3: GND -> /MCU/3V3
- JP8 pad 1: /MCU/3V3 -> GND
- JP8 pad 3: GND -> /MCU/3V3
- Q4 pad 1: /Motor/5V -> /Motor/Motor_Actuators/5V_ROBOTIS
- Q5 pad 1: /Motor/5V -> /Motor/Motor_Actuators/5V_ROBOTIS
- R47 pad 1: /Motor/5V -> /Motor/Motor_Actuators/5V_ROBOTIS
- R49 pad 1: /Motor/5V -> /Motor/Motor_Actuators/5V_ROBOTIS
- R50 pad 1: /Motor/5V -> /Motor/Motor_Actuators/5V_ROBOTIS
Routing:
- net /Power/Vbatt: track 0.00 -> 118.1 mm, vias 0 -> 1
- net /Motor/5V: track 0.00 -> 98.2 mm, vias 0 -> 1
- net /Motor/Motor_Actuators/Motor1_Low: track 0.00 -> 71.9 mm, vias 0 -> 2
- net /Motor/Motor_Actuators/Motor2_High: track 0.00 -> 64.7 mm, vias 0 -> 1
- net /Motor/Motor_Actuators/Motor2_Low: track 0.00 -> 62.0 mm, vias 0 -> 1
- net /Power/12V: track 0.00 -> 59.8 mm
- net /Motor/Motor_Actuators/Motor1_High: track 0.00 -> 59.5 mm, vias 0 -> 1
- net /MCU/3V3: track 0.00 -> 56.5 mm, vias 0 -> 16
- net /Power/Power_Buck_5V_Actuators/ENABLE: track 0.00 -> 45.2 mm, vias 0 -> 2
- net /MCU/MCU_Core/NRST: track 0.00 -> 44.5 mm, vias 0 -> 1
- net Net-(J13-TRIM(OPTIONAL)): track 0.00 -> 35.2 mm
- net Net-(J14-TRIM(OPTIONAL)): track 0.00 -> 34.4 mm
- net /Power/Power_Buck_12V/ENABLE: track 0.00 -> 28.9 mm
- net Net-(PS1-TRIM(OPTIONAL)): track 0.00 -> 26.0 mm
- net GND: track 0.00 -> 23.7 mm, vias 0 -> 17
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- added copper zone on F.Cu, net /MCU/5V_PC_EMBARQUE
- added copper zone on F.Cu, net /Motor/5V
- added copper zone on F.Cu, net /Motor/Motor_Actuators/PWR_5
- added copper zone on F.Cu, net /Power/12V
- added copper zone on F.Cu, net /Power/Power_Buck_12V/IN
- added copper zone on F.Cu, net /Power/Power_Buck_5V_Actuators/IN
- added copper zone on F.Cu, net /Power/Power_Buck_5V_Compute/IN
- added copper zone on F.Cu, net Net-(D3-K)
- added copper zone on F.Cu, net Net-(J12-Pin_2)
- added copper zone on F.Cu, net Net-(J4-Shield)
- added copper zone on In2.Cu, net Net-(J4-Shield)
Other:
- board text added: "5V"
- board text added: "LEFT ENCODER"
- board text added: "PCB Edge"
- board text added: "PRI MOTOR 1"
- board text added: "PRI MOTOR 2"
- board text added: "RIGHT ENCODER"
- board text added: "RX"
- board text added: "SEC MOTOR 1"
- board text added: "SEC MOTOR 2"
- board text added: "TRIM 12V"
- board text added: "TRIM 5V ACTUATOR"
- board text added: "TRIM 5V COMPUTE"
- board text added: "TX"

Commit message: continue
Parts:
- added C130: 10uF, Capacitor_SMD:C_0603_1608Metric_Pad1.08x0.95mm_HandSolder, F.Cu at (140.9, 132.8)
- added C131: 10uF, Capacitor_SMD:C_0603_1608Metric_Pad1.08x0.95mm_HandSolder, F.Cu at (129.9, 132.8)
- C105, C115, C116, C23, C24, C25, C26, C27, C28, C29, C30, C31, C32, C33, C34, C35, D1, D17, D18, D19, D2, D20, D21, FB2, IC2, IC3, IC4, IC9, J2, J3, J4, JP11, JP4, JP5, Q4, Q5, R10, R11, R12, R13, R14, R15, R16, R17, R18, R19, R2, R20, R21, R22, R23, R24, R25, R26, R27, R28, R29, R3, R4, R47, R48, R49, R5, R50, R55, R56, R57, R58, R59, R6, R7, R8, R9, T1, TP1, TP2, U1, U7, Y2: moved to B.Cu
- C106: value 100nF -> 10uF
- C107: value 100uF -> 10uF; footprint SamacSys_Parts:CAPAE830X1050N -> Capacitor_SMD:C_0603_1608Metric_Pad1.08x0.95mm_HandSolder
- moved D21 297.9 mm to (196.0, -45.3)
- moved R59 297.2 mm to (200.0, -45.0)
- moved D20 292.7 mm to (196.0, -42.8)
- moved R58 292.2 mm to (200.0, -42.5)
- moved D19 287.5 mm to (196.0, -40.2)
- moved R57 287.1 mm to (200.0, -40.0)
- moved D18 282.4 mm to (196.0, -37.6)
- moved R56 282.1 mm to (200.0, -37.5)
- moved D17 277.2 mm to (196.0, -35.0)
- moved R55 277.1 mm to (200.0, -34.9)
- moved IC2 272.7 mm to (187.0, -40.5)
- moved J4 259.0 mm to (150.7, 13.9)
- moved C35 257.2 mm to (143.5, 14.8), turned to -90 degrees
- moved R29 257.2 mm to (141.9, 14.8), turned to 90 degrees
- moved D2 256.9 mm to (145.1, 15.0), turned to 90 degrees
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Routing:
- net /Power/24V: track 0.00 -> 15.0 mm
- net /Motor/Motor_Actuators/PWR_2: track 0.00 -> 4.82 mm
- net /Motor/Motor_Actuators/PWR_3: track 0.00 -> 4.82 mm
- net /Motor/Motor_Actuators/PWR_4: track 0.00 -> 4.82 mm
- net /Motor/Motor_Actuators/PWR_1: track 0.00 -> 4.81 mm
- net Net-(D7-K): track 0.00 -> 1.60 mm
- added copper zone on F.Cu, net /Power/24V
- added copper zone on B.Cu, net Net-(J4-Shield)
- removed copper zone on F.Cu, net Net-(J4-Shield)
