File: Robot WallA/Robot WallA.kicad_pcb (KiCad board)
At the start: 4 copper layers, 170 x 100 mm, 312 parts, among them IC1 STM32F407IGT6, IC2 DS04-254-2-04BK-SMT, IC3 USBLC6-4SC6, IC4 USBLC6-4SC6, IC6 TLV75533PDBVR, IC7 ABXS005A4X341-SRZ, IC8 DRV8262DDVR, IC9 74LVC2G241DP-Q100H, J1 Conn_02x05_Female, J10 Conn_01x02, J11 Conn_01x02, J12 Conn_01x02, J13 NID35-5, J14 NID35-5, J15 39501-1002, J16 39501-1002, J17 39501-1004, J18 39501-1004, J19 22-03-5035, J2 USB4216-03-A, J20 22-03-5035, J21 22-03-5035, J22 22-03-5035, J23 Conn_01x03, J24 281695-3, J25 Conn_01x03, J26 281695-3, J27 Conn_01x03, J28 281695-3, J29 Conn_01x03, J3 SS-90000-009, J30 39501-1002, J31 39501-1002, J32 Conn_01x03, J33 281695-3, J34 Conn_01x03, J35 BM04B-SRSS-TB, J36 BM04B-SRSS-TB, J37 BM04B-SRSS-TB, J38 BM02B-SRSS-TB, J39 Conn_01x03, J4 USB_B_Micro, J40 BM03B-SRSS-TB, J41 BM03B-SRSS-TB, J42 BM03B-SRSS-TB, J43 BM03B-SRSS-TB, J44 BM02B-SRSS-TB, J45 BM04B-SRSS-TB, J46 BM02B-SRSS-TB, J47 BM02B-SRSS-TB, J6 Conn_02x36_Counter_Clockwise, J7 Conn_01x02, J8 XT90PW_M, J9 Conn_01x02, Q1 BSS138, Q2 BSS138, Q3 BSS138, Q4 BSS119, Q5 BSS119, SW1 Switch, T1 H1102NL, U1 FT231XS, U2 125700D00000G, U3 125700D00000G, U4 125700D00000G, U5 125700D00000G, U6 L298N, U7 LAN8742A, Y1 Crystal_GND24, Y2 Crystal_GND24

Commit message: Reworked 12V and 5V power supplies, continue routing
Parts:
- removed C126, C47, C48, C49: 4.7uF/50V, Capacitor_SMD:C_0805_2012Metric_Pad1.18x1.45mm_HandSolder
- removed C127, C50, C61: 10nF/50V, Capacitor_SMD:C_0805_2012Metric_Pad1.18x1.45mm_HandSolder
- removed C40: 120uF/25V, SamacSys_Parts:EEE0JA331XP
- removed C41, C42, C43: 47nF/25V, Capacitor_SMD:C_0603_1608Metric_Pad1.08x0.95mm_HandSolder
- removed C44, C45: 4.7uF/25V, Capacitor_SMD:C_1210_3225Metric_Pad1.33x2.70mm_HandSolder
- removed C46: 22uF/25V, SamacSys_Parts:EEE1AA220WR
- removed C97: 100uF/50V, SamacSys_Parts:CAPAE830X1050N
- removed J13, J14: NID35-5, SamacSys_Parts:NID355
- removed PS1, PS2: NID35-12, SamacSys_Parts:NID3512
- removed RV1: Trim 10k, SamacSys_Parts:TC33X2503E
- added D16: LED_RED, LED_SMD:LED_0603_1608Metric, F.Cu at (188.8, 61.5)
- added JP12: Closed, Jumper:SolderJumper-2_P1.3mm_Bridged_RoundedPad1.0x1.5mm, F.Cu at (179.1, 88.0)
- added JP13: Open, Jumper:SolderJumper-2_P1.3mm_Open_RoundedPad1.0x1.5mm, F.Cu at (176.4, 88.0)
- added JP14: Closed, Jumper:SolderJumper-2_P1.3mm_Bridged_RoundedPad1.0x1.5mm, F.Cu at (177.3, 61.3)
- added JP15: Open, Jumper:SolderJumper-2_P1.3mm_Open_RoundedPad1.0x1.5mm, F.Cu at (174.7, 61.3)
- added Q6: BSS138, Package_TO_SOT_SMD:SOT-23, F.Cu at (167.8, 88.3)
- added R53: 500R, Resistor_SMD:R_0603_1608Metric_Pad0.98x0.95mm_HandSolder, F.Cu at (145.2, 71.8)
- added R54: 21k, Resistor_SMD:R_0603_1608Metric_Pad0.98x0.95mm_HandSolder, F.Cu at (173.2, 86.9)
- added R60: 10k, Resistor_SMD:R_0603_1608Metric_Pad0.98x0.95mm_HandSolder, F.Cu at (167.8, 91.1)
- added RV4: Trim 2k, SamacSys_Parts:TC42X2202E, F.Cu at (148.3, 71.3)
- added U10: PTN78060W_EUW-7, Module:Texas_EUW_R-PDSS-T7_THT, F.Cu at (161.2, 44.7)
- added U8: PTN78020W, Module:Texas_EUK_R-PDSS-T7_THT, F.Cu at (122.8, 88.7)
- added U9: PTN78060W_EUW-7, Module:Texas_EUW_R-PDSS-T7_THT, F.Cu at (162.9, 71.2)
- C101, C102, C103, C104, C106, C107, C128, C129, C130, C131, C95, C96, C98, C99, J34, J35, J36, J37, J38, J39, J40, J41, J42, J43, J44, J45, J46, J47, J6: moved to B.Cu
- C105, IC9, Q4, Q5, R26, R47, R48, R49, R50, TP1, TP2: moved to F.Cu
- C117: value 120uF/25V -> 4.7uF/25V; footprint SamacSys_Parts:EEE0JA331XP -> Capacitor_SMD:C_1210_3225Metric_Pad1.33x2.70mm_HandSolder
- C118, C52, C53, C85: value 47nF/25V -> 4.7uF/50V; footprint Capacitor_SMD:C_0603_1608Metric_Pad1.08x0.95mm_HandSolder -> Capacitor_SMD:C_1210_3225Metric_Pad1.33x2.70mm_HandSolder
- C119, C54: value 47nF/25V -> 10nF/50V; footprint Capacitor_SMD:C_0603_1608Metric_Pad1.08x0.95mm_HandSolder -> Capacitor_SMD:C_0805_2012Metric_Pad1.18x1.45mm_HandSolder
- C120: value 47nF/25V -> 2.2uF/50V; footprint Capacitor_SMD:C_0603_1608Metric_Pad1.08x0.95mm_HandSolder -> Capacitor_SMD:C_1210_3225Metric_Pad1.33x2.70mm_HandSolder
- C121, C122, C56: value 4.7uF/25V -> 47nF/25V; footprint Capacitor_SMD:C_1210_3225Metric_Pad1.33x2.70mm_HandSolder -> Capacitor_SMD:C_0603_1608Metric_Pad1.08x0.95mm_HandSolder
- C123, C57, C89: value 22uF/25V -> 47nF/25V; footprint SamacSys_Parts:EEE1AA220WR -> Capacitor_SMD:C_0603_1608Metric_Pad1.08x0.95mm_HandSolder
- C124, C125, C59, C60: value 4.7uF/50V -> 4.7uF/25V; footprint Capacitor_SMD:C_0805_2012Metric_Pad1.18x1.45mm_HandSolder -> Capacitor_SMD:C_1210_3225Metric_Pad1.33x2.70mm_HandSolder
- C51: value 120uF/25V -> 330uF; footprint SamacSys_Parts:EEE0JA331XP -> SamacSys_Parts:CAPPRD500W65D1000H1800
- C55: value 4.7uF/25V -> 2.2uF/50V
- C58, C91, C92: value 4.7uF/50V -> 47nF/25V; footprint Capacitor_SMD:C_0805_2012Metric_Pad1.18x1.45mm_HandSolder -> Capacitor_SMD:C_0603_1608Metric_Pad1.08x0.95mm_HandSolder
- C83: value 120uF/25V -> 4.7uF/50V; footprint SamacSys_Parts:EEE0JA331XP -> Capacitor_SMD:C_1210_3225Metric_Pad1.33x2.70mm_HandSolder
- C84, C86: value 47nF/25V -> 330uF; footprint Capacitor_SMD:C_0603_1608Metric_Pad1.08x0.95mm_HandSolder -> SamacSys_Parts:CAPPRD500W65D1000H1800
- C87: value 4.7uF/25V -> 4.7uF/50V
- C88: value 4.7uF/25V -> 10nF/50V; footprint Capacitor_SMD:C_1210_3225Metric_Pad1.33x2.70mm_HandSolder -> Capacitor_SMD:C_0805_2012Metric_Pad1.18x1.45mm_HandSolder
- C90: value 4.7uF/50V -> 2.2uF/50V; footprint Capacitor_SMD:C_0805_2012Metric_Pad1.18x1.45mm_HandSolder -> Capacitor_SMD:C_1210_3225Metric_Pad1.33x2.70mm_HandSolder
- C93: value 10nF/50V -> 4.7uF/25V; footprint Capacitor_SMD:C_0805_2012Metric_Pad1.18x1.45mm_HandSolder -> Capacitor_SMD:C_1210_3225Metric_Pad1.33x2.70mm_HandSolder
- R31: value 100k -> 1.6k
- R32: value 10k -> 21k
- R40: value 100k -> 10k
- RV2, RV3: value Trim 10k -> Trim 2k; footprint SamacSys_Parts:TC33X2503E -> SamacSys_Parts:TC42X2202E
- moved J42 223.0 mm to (67.6, 42.5), turned to 0 degrees
- moved J43 222.4 mm to (75.6, 42.5), turned to 0 degrees
- moved J41 219.6 mm to (58.8, 54.4)
- moved J47 216.1 mm to (59.0, 125.8)
- moved J46 209.8 mm to (59.0, 118.6)
- moved J40 209.8 mm to (58.7, 62.6)
- moved J44 203.9 mm to (59.0, 111.4)
- moved J38 198.8 mm to (59.0, 104.2)
- moved D17 194.0 mm to (199.3, 159.0)
- moved D18 194.0 mm to (199.3, 156.4)
- moved D19 194.0 mm to (199.3, 153.8)
- moved D20 194.0 mm to (199.3, 151.2)
- moved D21 194.0 mm to (199.3, 148.7)
- moved IC2 194.0 mm to (190.3, 153.5)
- moved R55 194.0 mm to (203.3, 159.1)
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Connections:
- C118 pad 1: /Power/Power_Buck_12V/IN -> /Motor/5V
- C119 pad 1: /Power/Power_Buck_12V/IN -> /Motor/5V
- C120 pad 1: /Power/Power_Buck_12V/IN -> /Power/Power_Buck_5V_Actuators/IN
- C121 pad 1: /Power/Power_Buck_12V/IN -> /Power/Power_Buck_5V_Actuators/IN
- C122 pad 1: /Power/Power_Buck_12V/IN -> /Power/Power_Buck_5V_Actuators/IN
- C123 pad 1: /Power/12V -> /Power/Power_Buck_5V_Actuators/IN
- C124 pad 1: /Power/12V -> /Power/Power_Buck_5V_Actuators/IN
- C125 pad 1: /Power/12V -> /Power/Power_Buck_5V_Actuators/IN
- C51 pad 1: /Power/Power_Buck_5V_Actuators/IN -> /MCU/5V_PC_EMBARQUE
- C52 pad 1: /Power/Power_Buck_5V_Actuators/IN -> /MCU/5V_PC_EMBARQUE
- C53 pad 1: /Power/Power_Buck_5V_Actuators/IN -> /MCU/5V_PC_EMBARQUE
- C54 pad 1: /Power/Power_Buck_5V_Actuators/IN -> /MCU/5V_PC_EMBARQUE
- C55 pad 1: /Power/Power_Buck_5V_Actuators/IN -> /Power/Power_Buck_5V_Compute/IN
- C56 pad 1: /Power/Power_Buck_5V_Actuators/IN -> /Power/Power_Buck_5V_Compute/IN
- C57 pad 1: /Motor/5V -> /Power/Power_Buck_5V_Compute/IN
- C58 pad 1: /Motor/5V -> /Power/Power_Buck_5V_Compute/IN
- C59 pad 1: /Motor/5V -> /Power/Power_Buck_5V_Compute/IN
- C60 pad 1: /Motor/5V -> /Power/Power_Buck_5V_Compute/IN
- C83 pad 1: /Power/Power_Buck_12V/IN -> /Power/12V
- C84 pad 1: /Power/Power_Buck_12V/IN -> /Power/12V
- C85 pad 1: /Power/Power_Buck_12V/IN -> /Power/12V
- C86 pad 1: /Power/Power_Buck_12V/IN -> /Motor/5V
- C87 pad 1: /Power/Power_Buck_12V/IN -> /Motor/5V
- C88 pad 1: /Power/Power_Buck_12V/IN -> /Power/12V
- C89 pad 1: /Power/12V -> /Power/Power_Buck_12V/IN
- C90 pad 1: /Power/12V -> /Power/Power_Buck_12V/IN
- C91 pad 1: /Power/12V -> /Power/Power_Buck_12V/IN
- C92 pad 1: /Power/12V -> /Power/Power_Buck_12V/IN
- C93 pad 1: /Power/12V -> /Power/Power_Buck_12V/IN
- IC8 pad 14: /Motor/Motor_WheelDriver/Motor1_Low -> /Motor/Motor_WheelDriver/Motor2_Low
- IC8 pad 15: /Motor/Motor_WheelDriver/Motor1_Low -> /Motor/Motor_WheelDriver/Motor2_Low
- IC8 pad 16: /Motor/Motor_WheelDriver/Motor1_Low -> /Motor/Motor_WheelDriver/Motor2_Low
- IC8 pad 17: /Motor/Motor_WheelDriver/Motor1_High -> /Motor/Motor_WheelDriver/Motor2_High
- IC8 pad 18: /Motor/Motor_WheelDriver/Motor1_High -> /Motor/Motor_WheelDriver/Motor2_High
- IC8 pad 19: /Motor/Motor_WheelDriver/Motor1_High -> /Motor/Motor_WheelDriver/Motor2_High
- IC8 pad 4: /Motor/Motor_WheelDriver/Motor2_High -> /Motor/Motor_WheelDriver/Motor1_High
- IC8 pad 5: /Motor/Motor_WheelDriver/Motor2_High -> /Motor/Motor_WheelDriver/Motor1_High
- IC8 pad 6: /Motor/Motor_WheelDriver/Motor2_High -> /Motor/Motor_WheelDriver/Motor1_High
- IC8 pad 7: /Motor/Motor_WheelDriver/Motor2_Low -> /Motor/Motor_WheelDriver/Motor1_Low
- IC8 pad 8: /Motor/Motor_WheelDriver/Motor2_Low -> /Motor/Motor_WheelDriver/Motor1_Low
- IC8 pad 9: /Motor/Motor_WheelDriver/Motor2_Low -> /Motor/Motor_WheelDriver/Motor1_Low
- J15 pad 1: /Motor/Motor_WheelDriver/Motor1_High -> /Motor/Motor_WheelDriver/Motor2_Low
- J15 pad 2: /Motor/Motor_WheelDriver/Motor1_Low -> /Motor/Motor_WheelDriver/Motor2_High
- J16 pad 1: /Motor/Motor_WheelDriver/Motor2_High -> /Motor/Motor_WheelDriver/Motor1_High
- J16 pad 2: /Motor/Motor_WheelDriver/Motor2_Low -> /Motor/Motor_WheelDriver/Motor1_Low
- Q1 pad 1: /Power/GPIO_ENABLE_POWER_SUPPLIES -> /Power/Power_Buck_5V_Compute/GPIO_ENABLE
- Q1 pad 3: /Power/Power_Buck_5V_Actuators/ENABLE -> Net-(Q1-D)
- Q3 pad 3: /Power/Power_Buck_12V/ENABLE -> Net-(Q3-D)
- R31 pad 1: /Motor/5V -> Net-(D16-K)
- R31 pad 2: /Power/Power_Buck_5V_Actuators/ENABLE -> GND
- R32 pad 1: /Power/GPIO_ENABLE_POWER_SUPPLIES -> /Power/Power_Buck_5V_Compute/TRIM
- R32 pad 2: GND -> Net-(JP14-B)
- R40 pad 1: /Power/12V -> /Power/Power_Buck_5V_Compute/GPIO_ENABLE
- R40 pad 2: /Power/Power_Buck_12V/ENABLE -> GND
- RV2 pad 1: /Motor/5V -> Net-(JP15-B)
- RV2 pad 2: Net-(J14-TRIM(OPTIONAL)) -> GND
- RV2 pad 3: GND -> unconnected-(RV2-Pad3)
- RV3 pad 1: /Power/12V -> Net-(JP13-B)
- RV3 pad 2: Net-(PS1-TRIM(OPTIONAL)) -> GND
- RV3 pad 3: GND -> unconnected-(RV3-Pad3)
Routing:
- net /Power/12V: track 59.8 -> 376.2 mm
- net /Motor/5V: track 98.2 -> 382.9 mm, vias 1 -> 3
- net /Sensors/Vcc: track 0.00 -> 55.6 mm
- net /Power/Power_Buck_5V_Actuators/ENABLE: track 45.2 -> 0.00 mm, vias 2 -> 0
- net /Power/24V: track 15.0 -> 55.8 mm, vias 0 -> 4
- net /Sensors/Vcc2: track 0.00 -> 35.8 mm
- net Net-(J13-TRIM(OPTIONAL)): track 35.2 -> 0.00 mm
- net Net-(J14-TRIM(OPTIONAL)): track 34.4 -> 0.00 mm
- net /Power/Power_Buck_12V/ENABLE: track 28.9 -> 0.00 mm
- net Net-(PS1-TRIM(OPTIONAL)): track 26.0 -> 0.00 mm
- net /Power/Vbatt: track 118.1 -> 136.6 mm
- net /Motor/Motor_WheelDriver/Motor1_High: track 0.00 -> 13.9 mm
- net /Motor/Motor_WheelDriver/Motor2_High: track 0.00 -> 13.1 mm
- net /Motor/Motor_WheelDriver/Motor1_Low: track 0.00 -> 13.1 mm
- net /Motor/Motor_WheelDriver/Motor2_Low: track 0.00 -> 13.1 mm
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- added copper zone on F.Cu, net /Motor/Motor_WheelDriver/Motor1_High
- added copper zone on F.Cu, net /Motor/Motor_WheelDriver/Motor1_Low
- added copper zone on F.Cu, net /Motor/Motor_WheelDriver/Motor2_High
- added copper zone on F.Cu, net /Motor/Motor_WheelDriver/Motor2_Low
- added copper zone on B.Cu, net /Power/24V
- added copper zone on In2.Cu, net GND
- removed copper zone on F.Cu, net /Power/Power_Buck_5V_Actuators/IN
- removed copper zone on F.Cu, net Net-(J12-Pin_2)
Other:
- board text added: "Alim 5V Condo mal dimensionnés"
- board text added: "Manque condo"
- board text added: "PRIMARY MOTOR 1"
- board text added: "PRIMARY MOTOR 2"
- board text added: "SECONDARY MOTOR 1"
- board text added: "SECONDARY MOTOR 2"
- board text removed: "PRI MOTOR 1"
- board text removed: "PRI MOTOR 2"
- board text removed: "SEC MOTOR 1"
- board text removed: "SEC MOTOR 2"

Commit message: Conitnue routing
Parts:
- removed C110: 100uF, SamacSys_Parts:CAPAE830X1050N
- removed J6: Conn_02x36_Counter_Clockwise, Connector_PinHeader_2.54mm:PinHeader_2x36_P2.54mm_Vertical
- added J5: M20-8762042, SamacSys_Parts:M208762042, B.Cu at (150.9, 153.8)
- added JP16: Closed, Jumper:SolderJumper-2_P1.3mm_Bridged_RoundedPad1.0x1.5mm, F.Cu at (209.4, 113.8)
- added JP17: Closed, Jumper:SolderJumper-2_P1.3mm_Bridged_RoundedPad1.0x1.5mm, F.Cu at (205.8, 113.8)
- moved Q4 30.8 mm to (208.8, 117.2), turned to 90 degrees
- moved Q5 28.5 mm to (205.2, 117.2), turned to 90 degrees
- moved R47 27.4 mm to (208.8, 120.0), turned to 0 degrees
- moved TP1 25.5 mm to (209.1, 122.7), turned to -90 degrees
- moved R49 24.9 mm to (205.2, 120.0), turned to 0 degrees
- moved TP2 23.9 mm to (207.0, 122.6), turned to -90 degrees
- moved R26 22.2 mm to (210.1, 126.2), turned to -90 degrees
- moved IC9 19.2 mm to (207.5, 126.5), turned to 90 degrees
- moved C105 18.0 mm to (204.9, 125.4), turned to -90 degrees
- moved R50 17.7 mm to (208.8, 130.0), turned to 180 degrees
- moved FB2 16.5 mm to (122.2, 75.7)
- moved R48 14.3 mm to (204.9, 128.8), turned to -90 degrees
- moved D6 11.9 mm to (100.1, 96.0)
- moved R33 11.9 mm to (100.1, 97.8)
- moved R9 6.90 mm to (134.6, 88.2)
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Connections:
- C27 pad 1: /MCU/MCU_Peripherals/Q+ -> /MCU/MCU_Core/ETH7
- IC1 pad 107: /MCU/MCU_Core/PG3 -> /MCU/SECONDARY_MOTOR2
- IC1 pad 108: /MCU/MCU_Core/PG4 -> /MCU/SECONDARY_MOTOR3
- IC1 pad 109: /MCU/MCU_Core/PG5 -> /MCU/SECONDARY_MOTOR4
- IC1 pad 110: /MCU/MCU_Core/PG6 -> /MCU/SECONDARY_MOTOR5
- IC1 pad 115: /MCU/SENSORS11 -> /MCU/ENCODER0
- IC1 pad 116: /MCU/SENSORS10 -> /MCU/ENCODER1
- IC1 pad 117: /MCU/SENSORS9 -> /MCU/SENSORS10
- IC1 pad 118: /MCU/SENSORS8 -> /MCU/SENSORS11
- IC1 pad 162: /MCU/ENCODER0 -> /MCU/SENSORS8
- IC1 pad 163: /MCU/ENCODER1 -> /MCU/SENSORS9
- IC1 pad 17: /MCU/MCU_Core/PF1 -> /MCU/WHEEL7
- IC1 pad 176: /MCU/MCU_Core/PI7 -> /MCU/SERVO2
- IC1 pad 18: /MCU/MCU_Core/PF2 -> /MCU/WHEEL6
- IC1 pad 40: /MCU/SERVO3 -> /MCU/MCU_Core/PA0
- IC1 pad 51: /MCU/MCU_Core/PA5 -> /MCU/SERVO3
- IC1 pad 58: /MCU/MCU_Core/PB2 -> /MCU/SENSORS15
- IC1 pad 59: /MCU/MCU_Core/PF11 -> /MCU/SENSORS14
- IC1 pad 60: /MCU/MCU_Core/PF12 -> /MCU/SENSORS13
- IC1 pad 63: /MCU/MCU_Core/PF13 -> /MCU/SENSORS12
- IC1 pad 64: /MCU/MCU_Core/PF14 -> /MCU/SENSORS7
- IC1 pad 65: /MCU/MCU_Core/PF15 -> /MCU/SENSORS6
- IC1 pad 66: /MCU/MCU_Core/PG0 -> /MCU/SENSORS5
- IC1 pad 67: /MCU/MCU_Core/PG1 -> /MCU/SENSORS4
- IC1 pad 94: /MCU/MCU_Core/PB14 -> /Power/GPIO_PGOOD
- IC1 pad 95: /MCU/MCU_Core/PB15 -> /Power/GPIO_ENABLE_POWER_SUPPLIES
- J17 pad 2: /MCU/ENCODER0 -> /MCU/ENCODER2
- J17 pad 3: /MCU/ENCODER1 -> /MCU/ENCODER3
- J18 pad 2: /MCU/ENCODER2 -> /MCU/ENCODER0
- J18 pad 3: /MCU/ENCODER3 -> /MCU/ENCODER1
- U7 pad 5: /MCU/MCU_Peripherals/Q+ -> /MCU/MCU_Core/ETH7
- Y2 pad 1: /MCU/MCU_Peripherals/Q+ -> /MCU/MCU_Core/ETH7
Routing:
- net /MCU/3V3: track 60.0 -> 394.1 mm, vias 18 -> 22
- net /MCU/SENSORS9: track 0.00 -> 190.1 mm, vias 0 -> 3
- net /MCU/SENSORS11: track 0.00 -> 179.1 mm, vias 0 -> 3
- net /MCU/SENSORS10: track 0.00 -> 177.8 mm, vias 0 -> 3
- net /MCU/SENSORS8: track 0.00 -> 177.1 mm, vias 0 -> 3
- net /MCU/SENSORS3: track 0.00 -> 174.8 mm, vias 0 -> 3
- net /MCU/SENSORS2: track 0.00 -> 167.1 mm, vias 0 -> 3
- net /MCU/SENSORS1: track 0.00 -> 162.0 mm, vias 0 -> 3
- net /MCU/SENSORS4: track 0.00 -> 156.5 mm, vias 0 -> 3
- net /MCU/SENSORS0: track 0.00 -> 152.4 mm, vias 0 -> 2
- net /MCU/SENSORS6: track 0.00 -> 150.9 mm, vias 0 -> 3
- net /MCU/SENSORS7: track 0.00 -> 149.2 mm, vias 0 -> 2
- net /MCU/MCU_Core/NRST: track 44.5 -> 192.3 mm
- net /MCU/SENSORS5: track 0.00 -> 145.4 mm, vias 0 -> 3
- net /MCU/SENSORS15: track 0.00 -> 137.4 mm, vias 0 -> 2
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- added copper zone on F.Cu, net /Power/Power_Buck_5V_Actuators/IN
- added copper zone on B.Cu, net GND
- added copper zone on F.Cu, net GND
- added copper zone on In1.Cu, net GND
- added copper zone on In1.Cu, net GNDPWR
- added copper zone on F.Cu, net Net-(J11-Pin_2)
- added copper zone on F.Cu, net Net-(J12-Pin_2)
- added copper zone on In1.Cu, net Net-(J4-Shield)
- removed copper zone on In2.Cu, net GND
- removed copper zone on In2.Cu, net GNDPWR
- removed copper zone on In2.Cu, net Net-(J4-Shield)
Other:
- board text added: "!!WARNING!! TYPE-C IS A POWER OUTPUT!"
