File: Robot WallA/Motor_WheelDriver.kicad_sch (KiCad schematic)
At the start: 21 parts, among them J12 39501-1002, J13 39501-1002, U6 125700D00000G, U7 125700D00000G

Commit message: Continued to link MCU pins, Added a sheet for servomotors and optional 2 DC motors.
Parts:
- removed AC2: DRV8262DDVR, SOP64P810X120-44N, symbol SamacSys:DRV8262DDVR
- added AC1: DRV8262DDVR, SOP64P810X120-44N, symbol SamacSys_new:DRV8262DDVR
- renumbered C79 to C75, C80 to C76, C81 to C77, C82 to C78, C83 to C79, C84 to C80, C85 to C81, HS3 to HS2, J12 to J23, J13 to J24, JP9 to JP6, JP10 to JP7, JP11 to JP8, R37 to R39, R38 to R40, U6 to U4, U7 to U5
Connections:
- net 24V: now also AC1.11 (VM_2), AC1.12 (VM_3), AC1.2 (VM_1), AC1.21 (VM_4)
- net 3V3: now also JP6.3 (B), AC1.33 (VREF1), AC1.34 (VREF2), AC1.42 (VCC); no longer JP6.1 (A)
- net CurrentSenseMotor1: now also AC1.36 (IPROPI1)
- net CurrentSenseMotor2: now also AC1.37 (IPROPI2)
- net DECAY: now also AC1.30 (DECAY)
- net GND: now also JP6.1 (A), AC1.1 (GND_1), AC1.10 (GND_3), AC1.13 (GND_4), AC1.20 (GND_5), AC1.3 (GND_2), AC1.39 (MODE1), AC1.44 (GND_6); no longer JP6.3 (B)
- net Motor1_High: now also AC1.17 (OUT1_1), AC1.18 (OUT1_2), AC1.19 (OUT1_3)
- net Motor1_Low: now also AC1.14 (OUT2_1), AC1.15 (OUT2_2), AC1.16 (OUT2_3)
- net Motor2_High: now also AC1.4 (OUT3_1), AC1.5 (OUT3_2), AC1.6 (OUT3_3)
- net Motor2_Low: now also AC1.7 (OUT4_1), AC1.8 (OUT4_2), AC1.9 (OUT4_3)
- net NFAULT: now also AC1.41 (NFAULT)
- net PWM1: now also AC1.26 (IN1)
- net PWM2: now also AC1.27 (IN2)
- net PWM3: now also AC1.28 (IN3)
- net PWM4: now also AC1.29 (IN4)
- net SLEEP: now also AC1.25 (NSLEEP)
- net TOFF: now also AC1.32 (TOFF)
- net VCP: now also AC1.22 (VCP)
- net at C75.1: now also AC1.23 (CPH)
- net at C75.2: now also AC1.24 (CPL)
- net at JP6.2 (C): now also AC1.38 (MODE2)
- net at R40.1: now also AC1.40 (OCPM)
Other:
- note added: "Default Configuration: OCPM = 1 --> Over Current Protection error = Retry MODE = 0 --> PH/EN mode Toff = 1 --> Waiting time between change = 16µs Decay = HZ --> Auto detect mode"
- note removed: "Default Configuration: OCPM = 1 --> Over Current Protection error = Retry MODE = 1 --> PWM mode Toff = 1 --> Waiting time between change = 16µs Decay = HZ --> Auto detect mode"

Commit message: Defined every footprints
Parts:
- C100: renamed from C75; value 0.1uF/X7R -> 100nF/50V; footprint CAPC2012X94N -> Capacitor_SMD:C_0603_1608Metric_Pad1.08x0.95mm_HandSolder; Arrow Part Number 0805DC104MAT2A -> (none); Arrow Price/Stock https://www.arrow.com/en/products/0805dc104mat2a/avx -> (none); Height 0.94 -> (none); Manufacturer_Name Kyocera AVX -> (none); Manufacturer_Part_Number 0805DC104MAT2A -> (none); Mouser Part Number 581-0805DC104MAT2A -> (none); Mouser Price/Stock https://www.mouser.com/Search/Refine.aspx?Keyword=581-0805D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 -> (none)
- C94: renamed from C77; value 0.1uF/X7R -> 100nF; footprint CAPC2012X94N -> Capacitor_SMD:C_0603_1608Metric_Pad1.08x0.95mm_HandSolder; Arrow Part Number 0805DC104MAT2A -> (none); Arrow Price/Stock https://www.arrow.com/en/products/0805dc104mat2a/avx -> (none); Height 0.94 -> (none); Manufacturer_Name Kyocera AVX -> (none); Manufacturer_Part_Number 0805DC104MAT2A -> (none); Mouser Part Number 581-0805DC104MAT2A -> (none); Mouser Price/Stock https://www.mouser.com/Search/Refine.aspx?Keyword=581-0805D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 -> (none)
- C95: renamed from C80; value 1uF -> 1uF/50V; footprint CAPC2012X94N -> Capacitor_SMD:C_0603_1608Metric_Pad1.08x0.95mm_HandSolder; Arrow Part Number 0805DC104MAT2A -> (none); Arrow Price/Stock https://www.arrow.com/en/products/0805dc104mat2a/avx -> (none); Height 0.94 -> (none); Manufacturer_Name Kyocera AVX -> (none); Manufacturer_Part_Number 0805DC104MAT2A -> (none); Mouser Part Number 581-0805DC104MAT2A -> (none); Mouser Price/Stock https://www.mouser.com/Search/Refine.aspx?Keyword=581-0805D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 -> (none)
- C96: renamed from C76; value 0.01 uF -> 10nF/50V; footprint CAPC2012X94N -> Capacitor_SMD:C_0603_1608Metric_Pad1.08x0.95mm_HandSolder; Arrow Part Number 0805DC104MAT2A -> (none); Arrow Price/Stock https://www.arrow.com/en/products/0805dc104mat2a/avx -> (none); Height 0.94 -> (none); Manufacturer_Name Kyocera AVX -> (none); Manufacturer_Part_Number 0805DC104MAT2A -> (none); Mouser Part Number 581-0805DC104MAT2A -> (none); Mouser Price/Stock https://www.mouser.com/Search/Refine.aspx?Keyword=581-0805D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 -> (none)
- C97: renamed from C78; value 100uF -> 100uF/50V; footprint CAPAE660X800N -> SamacSys_Parts:CAPAE830X1050N; Height 8 -> (none); Manufacturer_Name Nichicon -> (none); Manufacturer_Part_Number UCH1V101MCS1GS -> EDK107M050A9MAA; Mouser Part Number 647-UCH1V101MCS1GS -> (none); Mouser Price/Stock https://www.mouser.co.uk/ProductDetail/Nichicon/UCH1V101MCS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 -> (none)
- C98: renamed from C79; value 100uF -> 100uF/50V; footprint CAPAE660X800N -> SamacSys_Parts:CAPAE830X1050N; Height 8 -> (none); Manufacturer_Name Nichicon -> (none); Manufacturer_Part_Number UCH1V101MCS1GS -> EDK107M050A9MAA; Mouser Part Number 647-UCH1V101MCS1GS -> (none); Mouser Price/Stock https://www.mouser.co.uk/ProductDetail/Nichicon/UCH1V101MCS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 -> (none)
- C99: renamed from C81; value 100uF -> 100uF/50V; footprint CAPAE660X800N -> SamacSys_Parts:CAPAE830X1050N; Height 8 -> (none); Manufacturer_Name Nichicon -> (none); Manufacturer_Part_Number UCH1V101MCS1GS -> EDK107M050A9MAA; Mouser Part Number 647-UCH1V101MCS1GS -> (none); Mouser Price/Stock https://www.mouser.co.uk/ProductDetail/Nichicon/UCH1V101MCS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 -> (none)
- IC8: renamed from AC1; footprint SOP64P810X120-44N -> SamacSys_Parts:SOP64P810X120-44N; Height 1.2 -> (none); Manufacturer_Name Texas Instruments -> (none)
- J13: renamed from J23; footprint 395011002 -> SamacSys_Parts:395011002; Height 9.6 -> (none); Manufacturer_Name Molex -> (none); Mouser Part Number 538-39501-1002 -> (none); Mouser Price/Stock https://www.mouser.co.uk/ProductDetail/Molex/39501-1002?qs=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 -> (none)
- J14: renamed from J24; footprint 395011002 -> SamacSys_Parts:395011002; Height 9.6 -> (none); Manufacturer_Name Molex -> (none); Mouser Part Number 538-39501-1002 -> (none); Mouser Price/Stock https://www.mouser.co.uk/ProductDetail/Molex/39501-1002?qs=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 -> (none)
- JP6, JP7: footprint Jumper:SolderJumper-3_P1.3mm_Bridged12_RoundedPad1.0x1.5mm -> Jumper:SolderJumper-3_P1.3mm_Bridged12_Pad1.0x1.5mm
- JP8: value SolderJumper_3_Open -> SolderJumper; footprint (none) -> Jumper:SolderJumper-3_P1.3mm_Open_Pad1.0x1.5mm
- R39, R40, R41: footprint (none) -> Resistor_SMD:R_0603_1608Metric_Pad0.98x0.95mm_HandSolder
- R42: renamed from R43; footprint (none) -> Resistor_SMD:R_0603_1608Metric_Pad0.98x0.95mm_HandSolder
- R43: renamed from R42; value NC -> 100k; footprint (none) -> Resistor_SMD:R_0603_1608Metric_Pad0.98x0.95mm_HandSolder; now not fitted
- U4, U5: footprint 125700D00000G -> SamacSys_Parts:125700D00000G; Arrow Part Number 125700D00000G -> (none); Arrow Price/Stock https://www.arrow.com/en/products/125700d00000g/aavid-therm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 -> (none); Height 7.19 -> (none); Manufacturer_Name Aavid Thermalloy -> (none); Mouser Part Number 532-125700D00000G -> (none); Mouser Price/Stock https://www.mouser.co.uk/ProductDetail/Aavid/125700D00000G?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 -> (none)

Commit message: Updated USB UART converter, Linked telemeter sensors.
Updated components indicators
Parts:
- renumbered J13 to J15, J14 to J16, R39 to R42, R40 to R43, R41 to R44, R42 to R45, R43 to R46

Commit message: Continue to route
Parts:
- removed C98, C99: 100uF/50V, SamacSys_Parts:CAPAE830X1050N, symbol SamacSys_Parts:UCH1V101MCS1GS
- added C128, C129, C98, C99: 100nF/50V, Capacitor_SMD:C_0603_1608Metric_Pad1.08x0.95mm_HandSolder, symbol SamacSys_Parts:0805DC104MAT2A
Connections:
- net 24V: now also C128.1, C129.1, C98.1, C99.1
- net 3V3: now also JP7.3 (B), JP8.3 (B); no longer JP7.1 (A), JP8.1 (A)
- net GND: now also JP7.1 (A), JP8.1 (A), C128.2, C129.2, C98.2, C99.2; no longer JP7.3 (B), JP8.3 (B)
Other:
- moved on the sheet: C94, C95, C96, C97

Commit message: Reworked 12V and 5V power supplies, continue routing
Parts:
- removed C97: 100uF/50V, SamacSys_Parts:CAPAE830X1050N, symbol SamacSys_Parts:UCH1V101MCS1GS
Connections:
- net Motor1_High: now also IC8.4 (OUT3_1), IC8.5 (OUT3_2), IC8.6 (OUT3_3), J16.1; no longer IC8.17 (OUT1_1), IC8.18 (OUT1_2), IC8.19 (OUT1_3), J15.1
- net Motor1_Low: now also IC8.7 (OUT4_1), IC8.8 (OUT4_2), IC8.9 (OUT4_3), J16.2; no longer IC8.14 (OUT2_1), IC8.15 (OUT2_2), IC8.16 (OUT2_3), J15.2
- net Motor2_High: now also IC8.17 (OUT1_1), IC8.18 (OUT1_2), IC8.19 (OUT1_3), J15.2; no longer IC8.4 (OUT3_1), IC8.5 (OUT3_2), IC8.6 (OUT3_3), J16.1
- net Motor2_Low: now also IC8.14 (OUT2_1), IC8.15 (OUT2_2), IC8.16 (OUT2_3), J15.1; no longer IC8.7 (OUT4_1), IC8.8 (OUT4_2), IC8.9 (OUT4_3), J16.2
Other:
- note added: "ATTENTION!! Pour simplifier le routage, les phases du moteurs on été invérsées! Atention au câblage!"
- moved on the sheet: C128, C129, C96, C98, C99, J15, J16

Commit message: Corrected all DRC erros, added info on PCB
modified distance meter connectors to be horizontal
Parts:
- HS2: footprint (none) -> Library:374524B60023G
Changed lines of the file:
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@@
 		(exclude_from_sim no)
 		(in_bom yes)
-		(on_board no)
+		(on_board yes)
 		(dnp no)
 		(fields_autoplaced yes)
@@
 			)
 		)
-		(property "Footprint" ""
+		(property "Footprint" "Library:374524B60023G"
 			(at 58.7248 161.29 0)
 			(effects

Commit message: Updated fab files.
Other:
- company: (none) -> Socotec Monitoring
- title: (none) -> Robot Wall-A
Changed lines of the file:
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@@
 	(generator_version "9.0")
 	(paper "A4")
+	(title_block
+		(title "Robot Wall-A")
+		(date "2025-09-20")
+		(rev "v1.0")
+		(company "Socotec Monitoring")
+		(comment 1 "GDU")
+		(comment 2 "THO")
+	)
 	(rectangle
 		(start 151.13 88.9)
@@
 			)
 		)
+		(property "MPN" ""
+			(at 193.04 123.19 90)
+			(effects
+				(font
+					(size 1.27 1.27)
+				)
+				(hide yes)
+			)
+		)
 		(pin "2"
 		)
@@
 			)
 		)
+		(property "MPN" ""
+			(at 213.36 57.15 90)
+			(effects
+				(font
+					(size 1.27 1.27)
+				)
+				(hide yes)
+			)
+		)
 		(pin "2"
 		)
@@
 			)
 		)
+		(property "MPN" ""
+			(at 173.99 101.6 0)
+			(effects
+				(font
+					(size 1.27 1.27)
+				)
+				(hide yes)
+			)
+		)
 		(pin "1"
 		)
@@
 			)
 		)
+		(property "MPN" ""
+			(at 198.12 57.15 90)
+			(effects
+				(font
+					(size 1.27 1.27)
+				)
+				(hide yes)
+			)
+		)
 		(pin "2"
 		)
@@
 			)
 		)
+		(property "MPN" ""
+			(at 182.88 57.15 90)
+			(effects
+				(font
+					(size 1.27 1.27)
+				)
+				(hide yes)
+			)
+		)
 		(pin "2"
 		)
@@
 			)
 		)
+		(property "MPN" ""
+			(at 248.92 86.36 0)
+			(effects
+				(font
+					(size 1.27 1.27)
+				)
+				(hide yes)
+			)
+		)
 		(pin "1"
 		)
@@
 			)
 		)
+		(property "MPN" ""
+			(at 184.15 127 0)
+			(effects
+				(font
+					(size 1.27 1.27)
+				)
+				(hide yes)
+			)
+		)
 		(pin "1"
 		)
@@
 			)
 		)
+		(property "MPN" ""
+			(at 198.12 101.6 0)
+			(effects
+				(font
+					(size 1.27 1.27)
+				)
+				(hide yes)
+			)
+		)
 		(pin "1"
 		)
@@
 			)
 		)
+		(property "MPN" ""
+			(at 154.94 44.45 90)
+			(effects
+				(font
+					(size 1.27 1.27)
+				)
+				(hide yes)
+			)
+		)
 		(pin "2"
 		)
@@
 			)
 		)
+		(property "MPN" ""
+			(at 60.96 62.23 0)
+			(effects
+				(font
+					(size 1.27 1.27)
+				)
+				(hide yes)
+			)
+		)
 		(pin "8"
 		)
@@
 			)
 		)
+		(property "MPN" ""
+			(at 154.94 57.15 90)
+			(effects
+				(font
+					(size 1.27 1.27)
+				)
+				(hide yes)
+			)
+		)
 		(pin "2"
 		)
@@
 			)
 		)
+		(property "MPN" ""
+			(at 120.65 68.58 0)
+			(effects
+				(font
+					(size 1.27 1.27)
+				)
+				(hide yes)
+			)
+		)
 		(pin "1"
 		)
@@
 			)
 		)
+		(property "MPN" ""
+			(at 106.68 66.04 0)
+			(effects
+				(font
+					(size 1.27 1.27)
+				)
+				(hide yes)
+			)
+		)
 		(pin "1"
 		)
@@
 			)
 		)
+		(property "MPN" ""
+			(at 116.84 120.65 90)
+			(effects
+				(font
+					(size 1.27 1.27)
+				)
+				(hide yes)
+			)
+		)
 		(pin "2"
 		)
@@
 			)
 		)
+		(property "MPN" ""
+			(at 82.55 35.56 90)
+			(effects
+				(font
+					(size 1.27 1.27)
+				)
+				(hide yes)
+			)
+		)
 		(pin "2"
 		)
@@
 			)
 		)
+		(property "MPN" ""
+			(at 248.92 76.2 0)
+			(effects
+				(font
+					(size 1.27 1.27)
+				)
+				(hide yes)
+			)
+		)
 		(pin "1"
 		)
@@
 			)
 		)
+		(property "MPN" ""
+			(at 58.42 161.29 0)
+			(effects
+				(font
+					(size 1.27 1.27)
+				)
+				(hide yes)
+			)
+		)
 		(instances
 			(project "PCB"
@@
 			)
 		)
+		(property "MPN" ""
+			(at 128.27 77.47 90)
+			(effects
+				(font
+					(size 1.27 1.27)
+				)
+				(hide yes)
+			)
+		)
 		(pin "2"
 		)
@@
 			)
 		)
+		(property "MPN" ""
+			(at 49.53 147.32 0)
+			(effects
+				(font
+					(size 1.27 1.27)
+				)
+				(hide yes)
+			)
+		)
 		(pin "2"
 		)
@@
 			)
 		)
+		(property "MPN" ""
+			(at 193.04 146.05 90)
+			(effects
+				(font
+					(size 1.27 1.27)
+				)
+				(hide yes)
+			)
+		)
 		(pin "3"
 		)
@@
 			)
 		)
+		(property "MPN" ""
+			(at 168.91 57.15 90)
+			(effects
+				(font
+					(size 1.27 1.27)
+				)
+				(hide yes)
+			)
+		)
 		(pin "2"
 		)
@@
 				(hide yes)
 			)
+		)
+		(property "MPN" ""
+			(at 49.53 137.16 0)
+			(effects
+				(font
+					(size 1.27 1.27)
+				)
+				(hide yes)
+			)

Commit message: Added to BOM connectors and socket
Updated fab files
Parts:
- added N13, N14: Connecteurs, symbol Mechanical:Housing
Changed lines of the file:
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@@
-			)
-		)
-		(property "MPN" ""
-			(at 193.04 123.19 90)
-			(effects
-				(font
-					(size 1.27 1.27)
-				)
-				(hide yes)
 			)
 		)
@@
 			)
 		)
-		(property "MPN" ""
-			(at 213.36 57.15 90)
-			(effects
-				(font
-					(size 1.27 1.27)
-				)
-				(hide yes)
-			)
-		)
 		(pin "2"
 		)
@@
 			)
 		)
-		(property "MPN" ""
-			(at 173.99 101.6 0)
-			(effects
-				(font
-					(size 1.27 1.27)
-				)
-				(hide yes)
-			)
-		)
 		(pin "1"
 		)
@@
 			)
 		)
-		(property "MPN" ""
-			(at 198.12 57.15 90)
-			(effects
-				(font
-					(size 1.27 1.27)
-				)
-				(hide yes)
-			)
-		)
 		(pin "2"
 		)
@@
 			)
 		)
-		(property "MPN" ""
-			(at 182.88 57.15 90)
-			(effects
-				(font
-					(size 1.27 1.27)
-				)
-				(hide yes)
-			)
-		)
 		(pin "2"
 		)
@@
 			)
 		)
-		(property "MPN" ""
-			(at 248.92 86.36 0)
-			(effects
-				(font
-					(size 1.27 1.27)
-				)
-				(hide yes)
-			)
-		)
 		(pin "1"
 		)
@@
 			)
 		)
-		(property "MPN" ""
-			(at 184.15 127 0)
-			(effects
-				(font
-					(size 1.27 1.27)
-				)
-				(hide yes)
-			)
-		)
 		(pin "1"
 		)
@@
 			)
 		)
-		(property "MPN" ""
-			(at 198.12 101.6 0)
-			(effects
-				(font
-					(size 1.27 1.27)
-				)
-				(hide yes)
-			)
-		)
 		(pin "1"
 		)
@@
 				(path "/117fd49e-499d-4b54-b58c-f6b538ecca4a/a16960dc-56f6-4cf6-af27-6c174f94c7f8/f5447fcd-99de-4b78-91ff-861a713e68d1"
 					(reference "R45")
+					(unit 1)
+				)
+			)
+		)
+	)
+	(symbol
+		(lib_id "Mechanical:Housing")
+		(at 261.62 66.04 0)
+		(unit 1)
+		(exclude_from_sim no)
+		(in_bom yes)
+		(on_board no)
+		(dnp no)
+		(property "Reference" "N14"
+			(at 265.43 65.0874 0)
+			(effects
+				(font
+					(size 1.27 1.27)
+				)
+				(justify left)
+			)
+		)
+		(property "Value" "Connecteurs"
+			(at 265.43 67.6274 0)
+			(effects
+				(font
+					(size 1.27 1.27)
+				)
+				(justify left)
+			)
+		)
+		(property "Footprint" ""
+			(at 262.89 64.77 0)
+			(effects
+				(font
+					(size 1.27 1.27)
+				)
+				(hide yes)
+			)
+		)
+		(property "Datasheet" "~"
+			(at 262.89 64.77 0)
+			(effects
+				(font
+					(size 1.27 1.27)
+				)
+				(hide yes)
+			)
+		)
+		(property "Description" "Housing"
+			(at 261.62 66.04 0)
+			(effects
+				(font
+					(size 1.27 1.27)
+				)
+				(hide yes)
+			)
+		)
+		(property "Manufacturer_Part_Number" "39503-2002"
+			(at 261.62 66.04 0)
+			(effects
+				(font
+					(size 1.27 1.27)
+				)
+				(hide yes)
+			)
+		)
+		(instances
+			(project "Robot WallA"
+				(path "/117fd49e-499d-4b54-b58c-f6b538ecca4a/a16960dc-56f6-4cf6-af27-6c174f94c7f8/f5447fcd-99de-4b78-91ff-861a713e68d1"
+					(reference "N14")
 					(unit 1)
 				)
@@
 			)
 		)
-		(property "MPN" ""
-			(at 154.94 44.45 90)
-			(effects
-				(font
-					(size 1.27 1.27)
-				)
-				(hide yes)
-			)
-		)
 		(pin "2"
 		)
@@
 			)
 		)
-		(property "MPN" ""
-			(at 60.96 62.23 0)
-			(effects
-				(font
-					(size 1.27 1.27)
-				)
-				(hide yes)
-			)
-		)
 		(pin "8"
 		)
@@
 			)
 		)
-		(property "MPN" ""
-			(at 154.94 57.15 90)
-			(effects
-				(font
-					(size 1.27 1.27)
-				)
-				(hide yes)
-			)
-		)
 		(pin "2"
 		)
@@
 			)
 		)
-		(property "MPN" ""
-			(at 120.65 68.58 0)
-			(effects
-				(font
-					(size 1.27 1.27)
-				)
-				(hide yes)
-			)
-		)
 		(pin "1"
 		)
@@
 			)
 		)
-		(property "MPN" ""
-			(at 106.68 66.04 0)
-			(effects
-				(font
-					(size 1.27 1.27)
-				)
-				(hide yes)
-			)
-		)
 		(pin "1"
 		)
@@
 			)
 		)
-		(property "MPN" ""
-			(at 116.84 120.65 90)
-			(effects
-				(font
-					(size 1.27 1.27)
-				)
-				(hide yes)
-			)
-		)
 		(pin "2"
 		)
@@
 			)
 		)
-		(property "MPN" ""
-			(at 82.55 35.56 90)
-			(effects
-				(font
-					(size 1.27 1.27)
-				)
-				(hide yes)
-			)
-		)
 		(pin "2"
 		)
@@
 				(path "/117fd49e-499d-4b54-b58c-f6b538ecca4a/a16960dc-56f6-4cf6-af27-6c174f94c7f8/f5447fcd-99de-4b78-91ff-861a713e68d1"
 					(reference "C94")
+					(unit 1)
+				)
+			)
+		)
+	)
+	(symbol
+		(lib_id "Mechanical:Housing")
+		(at 261.62 57.15 0)
+		(unit 1)
+		(exclude_from_sim no)
+		(in_bom yes)
+		(on_board no)
+		(dnp no)
+		(property "Reference" "N13"
+			(at 265.43 56.1974 0)
+			(effects
+				(font
+					(size 1.27 1.27)
+				)
+				(justify left)
+			)
+		)
+		(property "Value" "Connecteurs"
+			(at 265.43 58.7374 0)
+			(effects
+				(font
+					(size 1.27 1.27)
+				)
+				(justify left)
+			)
+		)
+		(property "Footprint" ""
+			(at 262.89 55.88 0)
+			(effects
+				(font
+					(size 1.27 1.27)
+				)
+				(hide yes)
+			)
+		)
+		(property "Datasheet" "~"
+			(at 262.89 55.88 0)
+			(effects
+				(font
+					(size 1.27 1.27)
+				)
+				(hide yes)
+			)
+		)
+		(property "Description" "Housing"
+			(at 261.62 57.15 0)
+			(effects
+				(font
+					(size 1.27 1.27)
+				)
+				(hide yes)
+			)
+		)
+		(property "Manufacturer_Part_Number" "39503-2002"
+			(at 261.62 57.15 0)
+			(effects
+				(font
+					(size 1.27 1.27)
+				)
+				(hide yes)
+			)
+		)
+		(instances
+			(project "Robot WallA"
+				(path "/117fd49e-499d-4b54-b58c-f6b538ecca4a/a16960dc-56f6-4cf6-af27-6c174f94c7f8/f5447fcd-99de-4b78-91ff-861a713e68d1"
+					(reference "N13")
 					(unit 1)
 				)
@@
 			)
 		)
-		(property "MPN" ""
-			(at 248.92 76.2 0)
-			(effects
-				(font
-					(size 1.27 1.27)
-				)
-				(hide yes)
-			)
-		)
 		(pin "1"
 		)
@@
 			)
 		)
-		(property "MPN" ""
-			(at 58.42 161.29 0)
-			(effects
-				(font
-					(size 1.27 1.27)
-				)
-				(hide yes)
-			)
-		)
 		(instances
 			(project "PCB"
@@
 			)
 		)
-		(property "MPN" ""
-			(at 128.27 77.47 90)
-			(effects
-				(font
-					(size 1.27 1.27)
-				)
-				(hide yes)
-			)
-		)
 		(pin "2"
 		)
@@
 			)
 		)
-		(property "MPN" ""
-			(at 49.53 147.32 0)
-			(effects
-				(font
-					(size 1.27 1.27)
-				)
-				(hide yes)
-			)
-		)
 		(pin "2"
 		)
@@
 			)
 		)
-		(property "MPN" ""
-			(at 193.04 146.05 90)
-			(effects
-				(font
-					(size 1.27 1.27)
-				)
-				(hide yes)
-			)
-		)
 		(pin "3"
 		)
@@
 			)
 		)
-		(property "MPN" ""
-			(at 168.91 57.15 90)
-			(effects
-				(font
-					(size 1.27 1.27)
-				)
-				(hide yes)
-			)
-		)
 		(pin "2"
 		)
@@
 				(hide yes)
 			)
-		)
-		(property "MPN" ""
-			(at 49.53 137.16 0)
-			(effects
-				(font
-					(size 1.27 1.27)
-				)
-				(hide yes)
-			)
