File: Robot WallA/Power_Buck_12V.kicad_sch (KiCad schematic)
At the start: 17 parts, among them Q2 BSS138

Commit message: Continued to link MCU pins, Added a sheet for servomotors and optional 2 DC motors.
Parts:
- renumbered C7 to C82, C90 to C83, C91 to C84, C92 to C85, C93 to C86, C94 to C87, C95 to C88, C96 to C89, C97 to C90, C98 to C91, C99 to C92, Q2 to Q4, R1 to R44, R3 to R45, RV1 to RV2
Changed lines of the file:
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@@
+	)
+	(junction
+		(at 261.62 29.21)
+		(diameter 0)
+		(color 0 0 0 0)
 	)
 	(junction
@@
 	(wire
 		(pts
-			(xy 257.81 29.21) (xy 264.16 29.21)
+			(xy 257.81 29.21) (xy 261.62 29.21)
 		)
 		(stroke
@@
 		(pts
 			(xy 137.16 118.11) (xy 137.16 120.65)
+		)
+		(stroke
+			(width 0)
+			(type default)
+		)
+	)
+	(wire
+		(pts
+			(xy 261.62 29.21) (xy 264.16 29.21)
 		)
 		(stroke
@@
 		(dnp no)
 		(fields_autoplaced yes)
-		(property "Reference" "#PWR07"
+		(property "Reference" "#PWR097"
 			(at 31.75 63.5 0)
 			(effects
@@
 			(project "PCB"
 				(path "/117fd49e-499d-4b54-b58c-f6b538ecca4a/d5f4dab0-e2de-4083-971d-4b1eb9c8d4bb/e9458b63-d596-4321-86fd-ad5fcfcf494d"
-					(reference "#PWR07")
+					(reference "#PWR097")
 					(unit 1)
 				)
@@
 		(on_board yes)
 		(dnp no)
-		(property "Reference" "R3"
+		(property "Reference" "R45"
 			(at 228.6 120.65 90)
 			(effects
@@
 			(project "PCB"
 				(path "/117fd49e-499d-4b54-b58c-f6b538ecca4a/d5f4dab0-e2de-4083-971d-4b1eb9c8d4bb/e9458b63-d596-4321-86fd-ad5fcfcf494d"
-					(reference "R3")
+					(reference "R45")
 					(unit 1)
 				)
@@
 		(on_board yes)
 		(dnp no)
-		(property "Reference" "C95"
+		(property "Reference" "C88"
 			(at 201.676 54.61 0)
 			(effects
@@
 			(project "PCB"
 				(path "/117fd49e-499d-4b54-b58c-f6b538ecca4a/d5f4dab0-e2de-4083-971d-4b1eb9c8d4bb/e9458b63-d596-4321-86fd-ad5fcfcf494d"
-					(reference "C95")
+					(reference "C88")
 					(unit 1)
 				)
@@
 		(on_board yes)
 		(dnp no)
-		(property "Reference" "C7"
+		(property "Reference" "C82"
 			(at 34.036 53.34 0)
 			(effects
@@
 			(project "PCB"
 				(path "/117fd49e-499d-4b54-b58c-f6b538ecca4a/d5f4dab0-e2de-4083-971d-4b1eb9c8d4bb/e9458b63-d596-4321-86fd-ad5fcfcf494d"
-					(reference "C7")
+					(reference "C82")
 					(unit 1)
 				)
@@
 		(on_board yes)
 		(dnp no)
-		(property "Reference" "C94"
+		(property "Reference" "C87"
 			(at 92.456 53.34 0)
 			(effects
@@
 			(project "PCB"
 				(path "/117fd49e-499d-4b54-b58c-f6b538ecca4a/d5f4dab0-e2de-4083-971d-4b1eb9c8d4bb/e9458b63-d596-4321-86fd-ad5fcfcf494d"
-					(reference "C94")
+					(reference "C87")
 					(unit 1)
 				)
@@
 		(on_board yes)
 		(dnp no)
-		(property "Reference" "C99"
+		(property "Reference" "C92"
 			(at 252.476 54.61 0)
 			(effects
@@
 			(project "PCB"
 				(path "/117fd49e-499d-4b54-b58c-f6b538ecca4a/d5f4dab0-e2de-4083-971d-4b1eb9c8d4bb/e9458b63-d596-4321-86fd-ad5fcfcf494d"
-					(reference "C99")
+					(reference "C92")
 					(unit 1)
 				)
@@
 		(dnp no)
 		(fields_autoplaced yes)
-		(property "Reference" "RV1"
+		(property "Reference" "RV2"
 			(at 91.44 119.3799 0)
 			(effects
@@
 			(project "PCB"
 				(path "/117fd49e-499d-4b54-b58c-f6b538ecca4a/d5f4dab0-e2de-4083-971d-4b1eb9c8d4bb/e9458b63-d596-4321-86fd-ad5fcfcf494d"
-					(reference "RV1")
+					(reference "RV2")
 					(unit 1)
 				)
@@
 		(on_board yes)
 		(dnp no)
-		(property "Reference" "C92"
+		(property "Reference" "C85"
 			(at 68.326 53.34 0)
 			(effects
@@
 			(project "PCB"
 				(path "/117fd49e-499d-4b54-b58c-f6b538ecca4a/d5f4dab0-e2de-4083-971d-4b1eb9c8d4bb/e9458b63-d596-4321-86fd-ad5fcfcf494d"
-					(reference "C92")
+					(reference "C85")
 					(unit 1)
 				)
@@
 		(dnp no)
 		(fields_autoplaced yes)
-		(property "Reference" "#PWR031"
+		(property "Reference" "#PWR0101"
 			(at 130.81 128.27 0)
 			(effects
@@
 			(project "PCB"
 				(path "/117fd49e-499d-4b54-b58c-f6b538ecca4a/d5f4dab0-e2de-4083-971d-4b1eb9c8d4bb/e9458b63-d596-4321-86fd-ad5fcfcf494d"
-					(reference "#PWR031")
+					(reference "#PWR0101")
 					(unit 1)
 				)
@@
 		(dnp no)
 		(fields_autoplaced yes)
-		(property "Reference" "#PWR06"
+		(property "Reference" "#PWR0104"
 			(at 215.9 130.81 0)
 			(effects
@@
 			(project "PCB"
 				(path "/117fd49e-499d-4b54-b58c-f6b538ecca4a/d5f4dab0-e2de-4083-971d-4b1eb9c8d4bb/e9458b63-d596-4321-86fd-ad5fcfcf494d"
-					(reference "#PWR06")
+					(reference "#PWR0104")
 					(unit 1)
 				)
@@
 		(on_board yes)
 		(dnp no)
-		(property "Reference" "C91"
+		(property "Reference" "C84"
 			(at 59.436 53.34 0)
 			(effects
@@
 			(project "PCB"
 				(path "/117fd49e-499d-4b54-b58c-f6b538ecca4a/d5f4dab0-e2de-4083-971d-4b1eb9c8d4bb/e9458b63-d596-4321-86fd-ad5fcfcf494d"
-					(reference "C91")
+					(reference "C84")
 					(unit 1)
 				)
@@
 		(on_board yes)
 		(dnp no)
-		(property "Reference" "R1"
+		(property "Reference" "R44"
 			(at 219.456 100.584 0)
 			(effects
@@
 			(project "PCB"
 				(path "/117fd49e-499d-4b54-b58c-f6b538ecca4a/d5f4dab0-e2de-4083-971d-4b1eb9c8d4bb/e9458b63-d596-4321-86fd-ad5fcfcf494d"
-					(reference "R1")
+					(reference "R44")
 					(unit 1)
 				)
@@
 		(dnp no)
 		(fields_autoplaced yes)
-		(property "Reference" "#PWR032"
+		(property "Reference" "#PWR0102"
 			(at 130.81 130.81 0)
 			(effects
@@
 			(project "PCB"
 				(path "/117fd49e-499d-4b54-b58c-f6b538ecca4a/d5f4dab0-e2de-4083-971d-4b1eb9c8d4bb/e9458b63-d596-4321-86fd-ad5fcfcf494d"
-					(reference "#PWR032")
+					(reference "#PWR0102")
 					(unit 1)
 				)
@@
 		(on_board yes)
 		(dnp no)
-		(property "Reference" "C96"
+		(property "Reference" "C89"
 			(at 218.186 54.61 0)
 			(effects
@@
 			(project "PCB"
 				(path "/117fd49e-499d-4b54-b58c-f6b538ecca4a/d5f4dab0-e2de-4083-971d-4b1eb9c8d4bb/e9458b63-d596-4321-86fd-ad5fcfcf494d"
-					(reference "C96")
+					(reference "C89")
 					(unit 1)
 				)
@@
 		(on_board yes)
 		(dnp no)
-		(property "Reference" "C97"
+		(property "Reference" "C90"
 			(at 228.346 54.61 0)
 			(effects
@@
 			(project "PCB"
 				(path "/117fd49e-499d-4b54-b58c-f6b538ecca4a/d5f4dab0-e2de-4083-971d-4b1eb9c8d4bb/e9458b63-d596-4321-86fd-ad5fcfcf494d"
-					(reference "C97")
+					(reference "C90")
 					(unit 1)
 				)
@@
 		(dnp no)
 		(fields_autoplaced yes)
-		(property "Reference" "#PWR024"
+		(property "Reference" "#PWR099"
 			(at 130.81 87.63 0)
 			(effects
@@
 			(project "PCB"
 				(path "/117fd49e-499d-4b54-b58c-f6b538ecca4a/d5f4dab0-e2de-4083-971d-4b1eb9c8d4bb/e9458b63-d596-4321-86fd-ad5fcfcf494d"
-					(reference "#PWR024")
+					(reference "#PWR099")
 					(unit 1)
 				)
@@
 		(dnp no)
 		(fields_autoplaced yes)
-		(property "Reference" "#PWR030"
+		(property "Reference" "#PWR098"
 			(at 93.98 130.81 0)
 			(effects
@@
 			(project "PCB"
 				(path "/117fd49e-499d-4b54-b58c-f6b538ecca4a/d5f4dab0-e2de-4083-971d-4b1eb9c8d4bb/e9458b63-d596-4321-86fd-ad5fcfcf494d"
-					(reference "#PWR030")
+					(reference "#PWR098")
 					(unit 1)
 				)
@@
 		(dnp no)
 		(fields_autoplaced yes)
-		(property "Reference" "Q2"
+		(property "Reference" "Q4"
 			(at 212.09 114.2999 0)
 			(effects
@@
 			(project "PCB"
 				(path "/117fd49e-499d-4b54-b58c-f6b538ecca4a/d5f4dab0-e2de-4083-971d-4b1eb9c8d4bb/e9458b63-d596-4321-86fd-ad5fcfcf494d"
-					(reference "Q2")
+					(reference "Q4")
+					(unit 1)
+				)
+			)
+		)
+	)
+	(symbol
+		(lib_id "power:PWR_FLAG")
+		(at 261.62 29.21 0)
+		(unit 1)
+		(exclude_from_sim no)
+		(in_bom yes)
+		(on_board yes)
+		(dnp no)
+		(fields_autoplaced yes)
+		(property "Reference" "#FLG05"
+			(at 261.62 27.305 0)
+			(effects
+				(font
+					(size 1.27 1.27)
+				)
+				(hide yes)
+			)
+		)
+		(property "Value" "PWR_FLAG"
+			(at 261.62 24.13 0)
+			(effects
+				(font
+					(size 1.27 1.27)
+				)
+				(hide yes)
+			)
+		)
+		(property "Footprint" ""
+			(at 261.62 29.21 0)
+			(effects
+				(font
+					(size 1.27 1.27)
+				)
+				(hide yes)
+			)
+		)
+		(property "Datasheet" "~"
+			(at 261.62 29.21 0)
+			(effects
+				(font
+					(size 1.27 1.27)
+				)
+				(hide yes)
+			)
+		)
+		(property "Description" "Special symbol for telling ERC where power comes from"
+			(at 261.62 29.21 0)
+			(effects
+				(font
+					(size 1.27 1.27)
+				)
+				(hide yes)
+			)
+		)
+		(pin "1"
+		)
+		(instances
+			(project "Robot WallA"
+				(path "/117fd49e-499d-4b54-b58c-f6b538ecca4a/d5f4dab0-e2de-4083-971d-4b1eb9c8d4bb/e9458b63-d596-4321-86fd-ad5fcfcf494d"
+					(reference "#FLG05")
 					(unit 1)
 				)
@@
 		(dnp no)
 		(fields_autoplaced yes)
-		(property "Reference" "#PWR025"
+		(property "Reference" "#PWR0100"
 			(at 130.81 90.17 0)
 			(effects
@@
 			(project "PCB"
 				(path "/117fd49e-499d-4b54-b58c-f6b538ecca4a/d5f4dab0-e2de-4083-971d-4b1eb9c8d4bb/e9458b63-d596-4321-86fd-ad5fcfcf494d"
-					(reference "#PWR025")
+					(reference "#PWR0100")
 					(unit 1)
 				)
@@
 		(on_board yes)
 		(dnp no)
-		(property "Reference" "C93"
+		(property "Reference" "C86"
 			(at 82.296 53.34 0)
 			(effects
@@
 			(project "PCB"
 				(path "/117fd49e-499d-4b54-b58c-f6b538ecca4a/d5f4dab0-e2de-4083-971d-4b1eb9c8d4bb/e9458b63-d596-4321-86fd-ad5fcfcf494d"
-					(reference "C93")
+					(reference "C86")
 					(unit 1)
 				)
@@
 		(on_board yes)
 		(dnp no)
-		(property "Reference" "C98"
+		(property "Reference" "C91"
 			(at 238.506 54.61 0)
 			(effects
@@
 			(project "PCB"
 				(path "/117fd49e-499d-4b54-b58c-f6b538ecca4a/d5f4dab0-e2de-4083-971d-4b1eb9c8d4bb/e9458b63-d596-4321-86fd-ad5fcfcf494d"
-					(reference "C98")
+					(reference "C91")
 					(unit 1)
 				)
@@
 		(dnp no)
 		(fields_autoplaced yes)
-		(property "Reference" "#PWR027"
+		(property "Reference" "#PWR0103"
 			(at 199.39 64.77 0)
 			(effects
@@
 			(project "PCB"
 				(path "/117fd49e-499d-4b54-b58c-f6b538ecca4a/d5f4dab0-e2de-4083-971d-4b1eb9c8d4bb/e9458b63-d596-4321-86fd-ad5fcfcf494d"
-					(reference "#PWR027")
+					(reference "#PWR0103")
 					(unit 1)
 				)
@@
 		(on_board yes)
 		(dnp no)
-		(property "Reference" "C90"
+		(property "Reference" "C83"
 			(at 50.546 53.34 0)
 			(effects
@@
 			(project "PCB"
 				(path "/117fd49e-499d-4b54-b58c-f6b538ecca4a/d5f4dab0-e2de-4083-971d-4b1eb9c8d4bb/e9458b63-d596-4321-86fd-ad5fcfcf494d"
-					(reference "C90")
+					(reference "C83")
 					(unit 1)
 				)

Commit message: Defined every footprints
Parts:
- added D15: LED_RED, LED_SMD:LED_0603_1608Metric, symbol Device:LED
- added R52: 5.1k, Resistor_SMD:R_0603_1608Metric_Pad0.98x0.95mm_HandSolder, symbol Device:R
- C83: renamed from C82; value 120u/25V -> 120uF/25V; footprint (none) -> SamacSys_Parts:EEE0JA331XP; Manufacturer_Part_Number (none) -> EEE-FNV121XUP
- C84: renamed from C83; value 47n/25V -> 47nF/25V; footprint (none) -> Capacitor_SMD:C_0603_1608Metric_Pad1.08x0.95mm_HandSolder
- C85: renamed from C84; value 47n/25V -> 47nF/25V; footprint (none) -> Capacitor_SMD:C_0603_1608Metric_Pad1.08x0.95mm_HandSolder
- C86: renamed from C85; value 47n/25V -> 47nF/25V; footprint (none) -> Capacitor_SMD:C_0603_1608Metric_Pad1.08x0.95mm_HandSolder
- C87: renamed from C86; value 4.7u/25V -> 4.7uF/25V; footprint (none) -> Capacitor_SMD:C_1210_3225Metric_Pad1.33x2.70mm_HandSolder
- C88: renamed from C87; value 4.7u/25V -> 4.7uF/25V; footprint (none) -> Capacitor_SMD:C_1210_3225Metric_Pad1.33x2.70mm_HandSolder
- C89: renamed from C88; value 22u/25V -> 22uF/25V; footprint (none) -> Capacitor_SMD:C_0805_2012Metric_Pad1.18x1.45mm_HandSolder
- C90: renamed from C89; value 4.7u/50V -> 4.7uF/50V; footprint (none) -> Capacitor_SMD:C_0805_2012Metric_Pad1.18x1.45mm_HandSolder
- C91: renamed from C90; value 4.7u/50V -> 4.7uF/50V; footprint (none) -> Capacitor_SMD:C_0805_2012Metric_Pad1.18x1.45mm_HandSolder
- C92: renamed from C91; value 4.7u/50V -> 4.7uF/50V; footprint (none) -> Capacitor_SMD:C_0805_2012Metric_Pad1.18x1.45mm_HandSolder
- C93: renamed from C92; value 10n/100V -> 10nF/50V; footprint (none) -> Capacitor_SMD:C_0805_2012Metric_Pad1.18x1.45mm_HandSolder
- PS1, PS2: footprint NID3512 -> SamacSys_Parts:NID3512; Arrow Part Number NID35-12 -> (none); Arrow Price/Stock https://www.arrow.com/en/products/nid35-12/mean-well-enterp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 -> (none); Height 13 -> (none); Manufacturer_Name Mean Well -> (none); Mouser Part Number 709-NID35-12 -> (none); Mouser Price/Stock https://www.mouser.co.uk/ProductDetail/MEAN-WELL/NID35-12?q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 -> (none)
- R37: renamed from R44; footprint (none) -> Resistor_SMD:R_0603_1608Metric_Pad0.98x0.95mm_HandSolder
- R38: renamed from R45; footprint (none) -> Resistor_SMD:R_0603_1608Metric_Pad0.98x0.95mm_HandSolder
- RV3: renamed from RV2; value NC-Trim 10k -> Trim 10k; footprint (none) -> SamacSys_Parts:TC33X2503E
- renumbered Q4 to Q3
Connections:
- net GND: now also R52.2
- net OUT: now also D15.2 (A)
- new net: D15.1 (K), R52.1

Commit message: Updated USB UART converter, Linked telemeter sensors.
Updated components indicators
Parts:
- Q3: Manufacturer_Part_Number (none) -> BSS138
- RV3: Manufacturer_Part_Number (none) -> TC33X2503E
- renumbered D15 to D7, R52 to R39, R37 to R40, R38 to R41
Changed lines of the file:
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@@
 		(dnp no)
 		(fields_autoplaced yes)
-		(property "Reference" "#PWR076"
+		(property "Reference" "#PWR081"
 			(at 31.75 63.5 0)
 			(effects
@@
 			(project "PCB"
 				(path "/117fd49e-499d-4b54-b58c-f6b538ecca4a/d5f4dab0-e2de-4083-971d-4b1eb9c8d4bb/e9458b63-d596-4321-86fd-ad5fcfcf494d"
-					(reference "#PWR076")
+					(reference "#PWR081")
 					(unit 1)
 				)
@@
 		(on_board yes)
 		(dnp no)
-		(property "Reference" "R38"
+		(property "Reference" "R41"
 			(at 228.6 120.65 90)
 			(effects
@@
 			(project "PCB"
 				(path "/117fd49e-499d-4b54-b58c-f6b538ecca4a/d5f4dab0-e2de-4083-971d-4b1eb9c8d4bb/e9458b63-d596-4321-86fd-ad5fcfcf494d"
-					(reference "R38")
+					(reference "R41")
 					(unit 1)
 				)
@@
 		(dnp no)
 		(fields_autoplaced yes)
-		(property "Reference" "#PWR0125"
+		(property "Reference" "#PWR080"
 			(at 163.83 52.07 0)
 			(effects
@@
 			(project "Robot WallA"
 				(path "/117fd49e-499d-4b54-b58c-f6b538ecca4a/d5f4dab0-e2de-4083-971d-4b1eb9c8d4bb/e9458b63-d596-4321-86fd-ad5fcfcf494d"
-					(reference "#PWR0125")
+					(reference "#PWR080")
 					(unit 1)
 				)
@@
 			)
 		)
+		(property "Manufacturer_Part_Number" "TC33X2503E"
+			(at 93.98 120.65 0)
+			(effects
+				(font
+					(size 1.27 1.27)
+				)
+				(hide yes)
+			)
+		)
 		(pin "2"
 		)
@@
 		(dnp no)
 		(fields_autoplaced yes)
-		(property "Reference" "#PWR082"
+		(property "Reference" "#PWR087"
 			(at 130.81 128.27 0)
 			(effects
@@
 			(project "PCB"
 				(path "/117fd49e-499d-4b54-b58c-f6b538ecca4a/d5f4dab0-e2de-4083-971d-4b1eb9c8d4bb/e9458b63-d596-4321-86fd-ad5fcfcf494d"
-					(reference "#PWR082")
+					(reference "#PWR087")
 					(unit 1)
 				)
@@
 		(dnp no)
 		(fields_autoplaced yes)
-		(property "Reference" "#PWR081"
+		(property "Reference" "#PWR086"
 			(at 215.9 130.81 0)
 			(effects
@@
 			(project "PCB"
 				(path "/117fd49e-499d-4b54-b58c-f6b538ecca4a/d5f4dab0-e2de-4083-971d-4b1eb9c8d4bb/e9458b63-d596-4321-86fd-ad5fcfcf494d"
-					(reference "#PWR081")
+					(reference "#PWR086")
 					(unit 1)
 				)
@@
 		(on_board yes)
 		(dnp no)
-		(property "Reference" "R52"
+		(property "Reference" "R39"
 			(at 153.67 52.07 90)
 			(effects
@@
 			(project "Robot WallA"
 				(path "/117fd49e-499d-4b54-b58c-f6b538ecca4a/d5f4dab0-e2de-4083-971d-4b1eb9c8d4bb/e9458b63-d596-4321-86fd-ad5fcfcf494d"
-					(reference "R52")
+					(reference "R39")
 					(unit 1)
 				)
@@
 		(on_board yes)
 		(dnp no)
-		(property "Reference" "D15"
+		(property "Reference" "D7"
 			(at 143.51 49.53 0)
 			(effects
@@
 			(project "Robot WallA"
 				(path "/117fd49e-499d-4b54-b58c-f6b538ecca4a/d5f4dab0-e2de-4083-971d-4b1eb9c8d4bb/e9458b63-d596-4321-86fd-ad5fcfcf494d"
-					(reference "D15")
+					(reference "D7")
 					(unit 1)
 				)
@@
 		(on_board yes)
 		(dnp no)
-		(property "Reference" "R37"
+		(property "Reference" "R40"
 			(at 219.456 100.584 0)
 			(effects
@@
 			(project "PCB"
 				(path "/117fd49e-499d-4b54-b58c-f6b538ecca4a/d5f4dab0-e2de-4083-971d-4b1eb9c8d4bb/e9458b63-d596-4321-86fd-ad5fcfcf494d"
-					(reference "R37")
+					(reference "R40")
 					(unit 1)
 				)
@@
 		(dnp no)
 		(fields_autoplaced yes)
-		(property "Reference" "#PWR083"
+		(property "Reference" "#PWR088"
 			(at 130.81 130.81 0)
 			(effects
@@
 			(project "PCB"
 				(path "/117fd49e-499d-4b54-b58c-f6b538ecca4a/d5f4dab0-e2de-4083-971d-4b1eb9c8d4bb/e9458b63-d596-4321-86fd-ad5fcfcf494d"
-					(reference "#PWR083")
+					(reference "#PWR088")
 					(unit 1)
 				)
@@
 		(dnp no)
 		(fields_autoplaced yes)
-		(property "Reference" "#PWR078"
+		(property "Reference" "#PWR083"
 			(at 130.81 87.63 0)
 			(effects
@@
 			(project "PCB"
 				(path "/117fd49e-499d-4b54-b58c-f6b538ecca4a/d5f4dab0-e2de-4083-971d-4b1eb9c8d4bb/e9458b63-d596-4321-86fd-ad5fcfcf494d"
-					(reference "#PWR078")
+					(reference "#PWR083")
 					(unit 1)
 				)
@@
 		(dnp no)
 		(fields_autoplaced yes)
-		(property "Reference" "#PWR080"
+		(property "Reference" "#PWR085"
 			(at 93.98 130.81 0)
 			(effects
@@
 			(project "PCB"
 				(path "/117fd49e-499d-4b54-b58c-f6b538ecca4a/d5f4dab0-e2de-4083-971d-4b1eb9c8d4bb/e9458b63-d596-4321-86fd-ad5fcfcf494d"
-					(reference "#PWR080")
+					(reference "#PWR085")
 					(unit 1)
 				)
@@
 			)
 		)
+		(property "Manufacturer_Part_Number" "BSS138"
+			(at 218.44 115.57 0)
+			(effects
+				(font
+					(size 1.27 1.27)
+				)
+				(hide yes)
+			)
+		)
 		(pin "2"
 		)
@@
 		(dnp no)
 		(fields_autoplaced yes)
-		(property "Reference" "#PWR079"
+		(property "Reference" "#PWR084"
 			(at 130.81 90.17 0)
 			(effects
@@
 			(project "PCB"
 				(path "/117fd49e-499d-4b54-b58c-f6b538ecca4a/d5f4dab0-e2de-4083-971d-4b1eb9c8d4bb/e9458b63-d596-4321-86fd-ad5fcfcf494d"
-					(reference "#PWR079")
+					(reference "#PWR084")
 					(unit 1)
 				)
@@
 		(dnp no)
 		(fields_autoplaced yes)
-		(property "Reference" "#PWR077"
+		(property "Reference" "#PWR082"
 			(at 199.39 64.77 0)
 			(effects
@@
 			(project "PCB"
 				(path "/117fd49e-499d-4b54-b58c-f6b538ecca4a/d5f4dab0-e2de-4083-971d-4b1eb9c8d4bb/e9458b63-d596-4321-86fd-ad5fcfcf494d"
-					(reference "#PWR077")
-					(unit 1)
-				)
+					(reference "#PWR082")
+					(unit 1)
+				)

Commit message: Continue to route
Parts:
- added C117: 120uF/25V, SamacSys_Parts:EEE0JA331XP, symbol Device:C_Polarized
- added C118, C119, C120: 47nF/25V, Capacitor_SMD:C_0603_1608Metric_Pad1.08x0.95mm_HandSolder, symbol Device:C
- added C121, C122: 4.7uF/25V, Capacitor_SMD:C_1210_3225Metric_Pad1.33x2.70mm_HandSolder, symbol Device:C
- added C123: 22uF/25V, SamacSys_Parts:EEE1AA220WR, symbol Device:C_Polarized
- added C124, C125, C126: 4.7uF/50V, Capacitor_SMD:C_0805_2012Metric_Pad1.18x1.45mm_HandSolder, symbol Device:C
- added C127: 10nF/50V, Capacitor_SMD:C_0805_2012Metric_Pad1.18x1.45mm_HandSolder, symbol Device:C
- C89: footprint Capacitor_SMD:C_0805_2012Metric_Pad1.18x1.45mm_HandSolder -> SamacSys_Parts:EEE1AA220WR; Height (none) -> 5.5; Manufacturer_Part_Number (none) -> EEE-FN1E220R
Connections:
- net GND: now also C117.2, C118.2, C119.2, C120.2, C121.2, C122.2, C123.2, C124.2, C125.2, C126.2, C127.2
- net IN: now also C117.1, C118.1, C119.1, C120.1, C121.1, C122.1
- net OUT: now also C123.1, C124.1, C125.1, C126.1, C127.1

Commit message: Reworked 12V and 5V power supplies, continue routing
Parts:
- removed C117, C83: 120uF/25V, SamacSys_Parts:EEE0JA331XP, symbol Device:C_Polarized
- removed C118, C119, C120, C84, C86: 47nF/25V, Capacitor_SMD:C_0603_1608Metric_Pad1.08x0.95mm_HandSolder, symbol Device:C
- removed C121, C122, C87: 4.7uF/25V, Capacitor_SMD:C_1210_3225Metric_Pad1.33x2.70mm_HandSolder, symbol Device:C
- removed C123, C89: 22uF/25V, SamacSys_Parts:EEE1AA220WR, symbol Device:C_Polarized
- removed C124, C125, C126: 4.7uF/50V, Capacitor_SMD:C_0805_2012Metric_Pad1.18x1.45mm_HandSolder, symbol Device:C
- removed C127: 10nF/50V, Capacitor_SMD:C_0805_2012Metric_Pad1.18x1.45mm_HandSolder, symbol Device:C
- removed PS1, PS2: NID35-12, SamacSys_Parts:NID3512, symbol SamacSys_new:NID35-12
- removed R40: 100k, Resistor_SMD:R_0603_1608Metric_Pad0.98x0.95mm_HandSolder, symbol Device:R
- removed RV3: Trim 10k, SamacSys_Parts:TC33X2503E, symbol Device:R_Potentiometer_Trim
- added C117: 4.7uF/25V, Capacitor_SMD:C_1210_3225Metric_Pad1.33x2.70mm_HandSolder, symbol Device:C
- added C83: 4.7uF/50V, Capacitor_SMD:C_1210_3225Metric_Pad1.33x2.70mm_HandSolder, symbol Device:C
- added C84: 330uF, SamacSys_Parts:CAPPRD500W65D1000H1800, symbol Device:C_Polarized
- added C89: 47nF/25V, Capacitor_SMD:C_0603_1608Metric_Pad1.08x0.95mm_HandSolder, symbol Device:C
- added R53: 500R, Resistor_SMD:R_0603_1608Metric_Pad0.98x0.95mm_HandSolder, symbol Device:R
- added RV4: Trim 2k, SamacSys_Parts:TC42X2202E, symbol Device:R_Potentiometer_Trim
- added U8: PTN78020W, Module:Texas_EUK_R-PDSS-T7_THT, symbol Converter_DCDC:PTN78020W_EUK-7
- C85: value 47nF/25V -> 4.7uF/50V; footprint Capacitor_SMD:C_0603_1608Metric_Pad1.08x0.95mm_HandSolder -> Capacitor_SMD:C_1210_3225Metric_Pad1.33x2.70mm_HandSolder; Manufacturer_Part_Number (none) -> GRM32ER71H475KA88L
- C88: value 4.7uF/25V -> 10nF/50V; footprint Capacitor_SMD:C_1210_3225Metric_Pad1.33x2.70mm_HandSolder -> Capacitor_SMD:C_0805_2012Metric_Pad1.18x1.45mm_HandSolder
- C90: value 4.7uF/50V -> 2.2uF/50V; footprint Capacitor_SMD:C_0805_2012Metric_Pad1.18x1.45mm_HandSolder -> Capacitor_SMD:C_1210_3225Metric_Pad1.33x2.70mm_HandSolder; Manufacturer_Part_Number (none) -> C3225X7R1H225K250AB
- C91, C92: value 4.7uF/50V -> 47nF/25V; footprint Capacitor_SMD:C_0805_2012Metric_Pad1.18x1.45mm_HandSolder -> Capacitor_SMD:C_0603_1608Metric_Pad1.08x0.95mm_HandSolder
- C93: value 10nF/50V -> 4.7uF/25V; footprint Capacitor_SMD:C_0805_2012Metric_Pad1.18x1.45mm_HandSolder -> Capacitor_SMD:C_1210_3225Metric_Pad1.33x2.70mm_HandSolder; Manufacturer_Part_Number (none) -> GRM32ER71H475KA88L
- R41: now not fitted
Connections:
- net GNDREF is gone; now on net GND: Q3.2 (S), R41.2
- net GND: now also C117.2, C83.2, C84.2, C89.2, RV4.2, U8.1 (GND), U8.7 (GND)
- net IN: now also C90.1, C91.1, C92.1, C93.1, C117.1, C89.1, U8.2 (VI); no longer C85.1, C88.1
- net OUT: now also C85.1, C88.1, C83.1, C84.1, U8.5 (VO_Sense), U8.6 (VO); no longer C90.1, C91.1, C92.1, C93.1
- net ENABLE: no longer names the net of Q3.3 (D)
- net ENABLE: now also U8.3 (~{Inhibit})
- new net: R53.2, RV4.1
- new net TRIM: R53.1, U8.4 (VO_Adj)
- no-connect marks 0 -> 1
Other:
- note removed: "footprint size 10n --> 0805 47n --> 0603 4,7uF --> 1210"
- moved on the sheet: C90, Q3
