File: Robot WallA/Power_Buck_12V.kicad_sch (KiCad schematic)
At the start: 17 parts, among them Q3 BSS138, U8 PTN78020W

Commit message: Modified footprint to simplify BOM. Finalized BOM.
Updated fab files
Parts:
- C117, C93: value 4.7uF/25V -> 4.7uF/50V
- C88: Manufacturer_Part_Number (none) -> CL21B103KBANNNC
- C89, C91, C92: value 47nF/25V -> 47nF/50V; Manufacturer_Part_Number (none) -> CC0603KPX7R9BB473
- R39: Manufacturer_Part_Number (none) -> CRCW06035K10FKEA
- R41: Manufacturer_Part_Number (none) -> 667-ERJ-3GEYJ103V
- R53: value 500R -> 549R; Manufacturer_Part_Number (none) -> RC0603FR-07549RL
