File: Robot WallA/Power.kicad_sch (KiCad schematic)
At the start: 25 parts, among them IC6 TLV75533PDBVR, J10 Conn_01x02, J11 Conn_01x02, J12 Conn_01x02, J7 Conn_01x02, J8 XT90PW_M, J9 Conn_01x02

Commit message: Added 3 thermistor to measure temperature near 12V and 24V power supplies and near motor drivers
Parts:
- removed J8: XT90PW_M, Connector_AMASS:AMASS_XT90PW-M_1x02_P10.90mm_Horizontal, symbol Connector_Generic:Conn_01x02
- added J8: XT90PW_M, Connector_AMASS:AMASS_XT90PW-M_1x02_P10.90mm_Horizontal, symbol Connector_Generic_MountingPin:Conn_02x01_MountingPin
- added R61: 10k, Resistor_SMD:R_0603_1608Metric_Pad0.98x0.95mm_HandSolder, symbol Device:R
- added TH1: Thermistor_NTC, Resistor_SMD:R_0603_1608Metric_Pad0.98x0.95mm_HandSolder, symbol Device:Thermistor_NTC
Connections:
- net 3V3: now also R61.2
- net GND: now also J8.1 (Pin_1), J8.MP (MountPin), TH1.2
- net Vbatt: now also J8.2 (Pin_2)
- new net ADC_POWER_SUPPLIES_TEMPERATURE: R61.1, TH1.1
Other:
- note added: "Mesure la température au milieu des Alimentations 12V et 24V"

Commit message: Modified footprint to simplify BOM. Finalized BOM.
Updated fab files
Parts:
- C36, C38: Manufacturer_Part_Number (none) -> CL10A106MA8NRNC
- C37, C39: Manufacturer_Part_Number (none) -> KGM15BR71H104KT
- J11, J12, J7: now left out of the parts list
- R61: Manufacturer_Part_Number (none) -> 667-ERJ-3GEYJ103V
